File: HW/KiCad/retro-001/retro-001.kicad_pcb (KiCad board)
At the start: 2 copper layers, 100 x 100 mm, 103 parts, among them J100 x, J101 x, J102 x, J103 x, J104 x, J105 x, J106 x, J21 x, J22 x, J37 x, J38 x, J39 x, J4 SysBus, J40 x, J41 x, J42 x, J43 x, J44 x, J45 x, J46 x, J47 x, J48 x, J49 x, J50 x, J51 x, J52 x, J53 x, J54 x, J55 x, J56 x, J57 x, J58 x, J59 x, J6 SysBus, J60 x, J61 x, J62 x, J63 x, J64 x, J65 x, J66 x, J67 x, J68 x, J69 x, J70 x, J71 x, J72 x, J73 x, J74 x, J75 x, J76 x, J77 x, J78 x, J79 x, J80 x, J81 x, J82 x, J83 x, J84 x, J85 x, J86 x, J87 x, J88 x, J89 x, J90 x, J91 x, J92 x, J93 x, J94 x, J95 x, J96 x, J97 x, J98 x, J99 x, M3 CY7C109D-10ZXI, U1 HD6309, U2 ATF1504AS-10AU100

Commit message: retro-002, mozna funkcni?
Parts:
- removed JTAG1: JTAG, Connector_IDC:IDC-Header_2x05_P2.54mm_Vertical
- added C12: 100n RESET, MHF:C_Disc_D3.0mm_W2.0mm_P2.50mm, F.Cu at (198.8, 43.8)
- added Cx19: 10p, MHF:C_Disc_D3.0mm_W2.0mm_P2.50mm, F.Cu at (220.0, 89.4)
- added Cx20: 10p, MHF:C_Disc_D3.0mm_W2.0mm_P2.50mm, F.Cu at (220.0, 86.9)
- added Cx21: 10p, MHF:C_Disc_D3.0mm_W2.0mm_P2.50mm, F.Cu at (220.0, 84.3)
- added Cx22: 10p, MHF:C_Disc_D3.0mm_W2.0mm_P2.50mm, F.Cu at (220.0, 81.8)
- added Cx23: 10p, MHF:C_Disc_D3.0mm_W2.0mm_P2.50mm, F.Cu at (217.2, 116.1)
- added Cx24: 10p, MHF:C_Disc_D3.0mm_W2.0mm_P2.50mm, F.Cu at (217.2, 113.5)
- added Cx25: 10p, MHF:C_Disc_D3.0mm_W2.0mm_P2.50mm, F.Cu at (217.2, 111.0)
- added Cx26: 10p, MHF:C_Disc_D3.0mm_W2.0mm_P2.50mm, F.Cu at (217.2, 108.5)
- added Cx27: Cx, MHF:CP_Radial_D5.0mm_P2.50mm, F.Cu at (166.4, 43.1)
- added Cx28: Cx, MHF:CP_Radial_D5.0mm_P2.50mm, F.Cu at (191.0, 60.9)
- added D2: D, MHF:D_1210_3225Metric_HandSolder, F.Cu at (180.3, 52.1)
- added J1: Conn_02x05_JTAG, Connector_IDC:IDC-Header_2x05_P2.54mm_Vertical, F.Cu at (215.7, 50.3)
- added J12: Reset, MHF:PinHole_1x01_2.54xrectangle, F.Cu at (196.2, 43.8)
- added J2: Conn_02x05_JTAG, Connector_IDC:IDC-Header_2x05_P2.54mm_Vertical, F.Cu at (172.5, 109.6)
- added J3: Serial, MHF:PinHeader_1x04_P2.54mm_Vertical, F.Cu at (237.5, 121.9)
- added J7: Conn_01x16_Pin, MHF:G_SOIC-16_3.9x9.9mm_HandSolder, B.Cu at (231.1, 55.8)
- added JP1: Nx4, MHF:SolderJumper-2_P1.3mm_Bridged_Pad1.0x1.5mm, B.Cu at (241.3, 109.4)
- added JP13: Nx3, MHF:SolderJumper-2_P1.3mm_Bridged_Pad1.0x1.5mm, B.Cu at (225.5, 112.8)
- added JP2: Nx5, MHF:SolderJumper-2_P1.3mm_Bridged_Pad1.0x1.5mm, B.Cu at (241.3, 113.2)
- added JP3: Nx6, MHF:SolderJumper-2_P1.3mm_Bridged_Pad1.0x1.5mm, B.Cu at (241.3, 116.2)
- added Jx1: BugFix, MHF:PinHeader_1x03_P2.54mm_Vertical, F.Cu at (241.9, 43.2)
- added Jx4: J, MHF:PinHeader_1x08_P2.54mm_Vertical, F.Cu at (250.2, 84.5)
- added L0: A0, MHF:LED_0805_2012Metric, F.Cu at (170.2, 28.0)
- added L1: A0, MHF:LED_0805_2012Metric, F.Cu at (172.7, 28.0)
- added L10: A0, MHF:LED_0805_2012Metric, F.Cu at (194.3, 27.9)
- added L11: A0, MHF:LED_0805_2012Metric, F.Cu at (196.8, 27.9)
- added L12: A0, MHF:LED_0805_2012Metric, F.Cu at (199.4, 27.9)
- added L13: A0, MHF:LED_0805_2012Metric, F.Cu at (201.9, 27.9)
- added L14: A0, MHF:LED_0805_2012Metric, F.Cu at (204.5, 27.9)
- added L15: A0, MHF:LED_0805_2012Metric, F.Cu at (207.0, 27.9)
- added L16: A0, MHF:LED_0805_2012Metric, F.Cu at (210.8, 27.9)
- added L17: A0, MHF:LED_0805_2012Metric, F.Cu at (213.4, 27.9)
- added L18: A0, MHF:LED_0805_2012Metric, F.Cu at (215.9, 27.9)
- added L19: A0, MHF:LED_0805_2012Metric, F.Cu at (218.4, 27.9)
- added L2: A0, MHF:LED_0805_2012Metric, F.Cu at (175.3, 28.0)
- added L20: A0, MHF:LED_0805_2012Metric, F.Cu at (221.0, 27.9)
- added L21: A0, MHF:LED_0805_2012Metric, F.Cu at (223.5, 27.9)
- added L22: A0, MHF:LED_0805_2012Metric, F.Cu at (226.1, 27.9)
- added L23: A0, MHF:LED_0805_2012Metric, F.Cu at (228.6, 27.9)
- added L24: A0, MHF:LED_0805_2012Metric, F.Cu at (165.1, 121.9)
- added L25: A0, MHF:LED_0805_2012Metric, F.Cu at (167.6, 121.9)
- added L26: A0, MHF:LED_0805_2012Metric, F.Cu at (170.2, 121.9)
- added L27: A0, MHF:LED_0805_2012Metric, F.Cu at (172.7, 121.9)
- added L28: A0, MHF:LED_0805_2012Metric, F.Cu at (175.3, 121.9)
- added L29: A0, MHF:LED_0805_2012Metric, F.Cu at (177.8, 121.9)
- added L3: A0, MHF:LED_0805_2012Metric, F.Cu at (177.8, 28.0)
- added L30: A0, MHF:LED_0805_2012Metric, F.Cu at (182.9, 121.9)
- added L31: A0, MHF:LED_0805_2012Metric, F.Cu at (185.4, 121.9)
- added L32: A0, MHF:LED_0805_2012Metric, F.Cu at (190.5, 121.9)
- added L33: A0, MHF:LED_0805_2012Metric, F.Cu at (193.0, 121.9)
- added L34: A0, MHF:LED_0805_2012Metric, F.Cu at (195.6, 121.9)
- added L35: A0, MHF:LED_0805_2012Metric, F.Cu at (198.1, 121.9)
- added L4: A0, MHF:LED_0805_2012Metric, F.Cu at (180.3, 28.0)
- added L5: A0, MHF:LED_0805_2012Metric, F.Cu at (182.9, 28.0)
- added L6: A0, MHF:LED_0805_2012Metric, F.Cu at (165.1, 27.9)
- added L7: A0, MHF:LED_0805_2012Metric, F.Cu at (167.6, 27.9)
- added L8: A0, MHF:LED_0805_2012Metric, F.Cu at (189.2, 27.9)
- added L9: A0, MHF:LED_0805_2012Metric, F.Cu at (191.8, 27.9)
- added LHALT1: A0, MHF:LED_0805_2012Metric, F.Cu at (215.9, 121.9)
- added LReset1: A0, MHF:LED_0805_2012Metric, F.Cu at (186.1, 31.8)
- added LS1: Speaker_Crystal, Buzzer_Beeper:MagneticBuzzer_Kingstate_KCG0601, F.Cu at (240.8, 29.3)
- added LSys1: A0, MHF:LED_0805_2012Metric, F.Cu at (195.3, 84.1)
- added PA1: J, MHF:PinHeader_1x10_P2.54mm_Vertical, F.Cu at (250.2, 112.4)
- added PB1: J, MHF:PinHeader_1x10_P2.54mm_Vertical, F.Cu at (250.2, 61.6)
- added Q1: MMBT3904, Package_TO_SOT_SMD:SOT-23, B.Cu at (233.0, 29.3)
- added R0: 1k, MHF:R_0805_2012Metric_Pad1.20x1.40mm_HandSolder, B.Cu at (170.2, 28.0)
- added R1: 1k, MHF:R_0805_2012Metric_Pad1.20x1.40mm_HandSolder, B.Cu at (172.7, 28.0)
- added R10: 1k, MHF:R_0805_2012Metric_Pad1.20x1.40mm_HandSolder, B.Cu at (194.3, 27.9)
- added R11: 1k, MHF:R_0805_2012Metric_Pad1.20x1.40mm_HandSolder, B.Cu at (196.8, 27.9)
- added R12: 1k, MHF:R_0805_2012Metric_Pad1.20x1.40mm_HandSolder, B.Cu at (199.4, 27.9)
- added R13: 1k, MHF:R_0805_2012Metric_Pad1.20x1.40mm_HandSolder, B.Cu at (201.9, 27.9)
- added R14: 1k, MHF:R_0805_2012Metric_Pad1.20x1.40mm_HandSolder, B.Cu at (204.5, 27.9)
- added R15: 1k, MHF:R_0805_2012Metric_Pad1.20x1.40mm_HandSolder, B.Cu at (207.0, 27.9)
- added R16: 1k, MHF:R_0805_2012Metric_Pad1.20x1.40mm_HandSolder, B.Cu at (210.8, 27.9)
- added R17: 1k, MHF:R_0805_2012Metric_Pad1.20x1.40mm_HandSolder, B.Cu at (213.4, 27.9)
- added R18: 1k, MHF:R_0805_2012Metric_Pad1.20x1.40mm_HandSolder, B.Cu at (215.9, 27.9)
- added R19: 1k, MHF:R_0805_2012Metric_Pad1.20x1.40mm_HandSolder, B.Cu at (218.4, 27.9)
- added R2: 1k, MHF:R_0805_2012Metric_Pad1.20x1.40mm_HandSolder, B.Cu at (175.3, 28.0)
- added R20: 1k, MHF:R_0805_2012Metric_Pad1.20x1.40mm_HandSolder, B.Cu at (221.0, 27.9)
- added R21: 1k, MHF:R_0805_2012Metric_Pad1.20x1.40mm_HandSolder, B.Cu at (223.5, 27.9)
- added R22: 1k, MHF:R_0805_2012Metric_Pad1.20x1.40mm_HandSolder, B.Cu at (226.1, 27.9)
- added R23: 1k, MHF:R_0805_2012Metric_Pad1.20x1.40mm_HandSolder, B.Cu at (228.6, 27.9)
- added R24: 1k, MHF:R_0805_2012Metric_Pad1.20x1.40mm_HandSolder, B.Cu at (165.1, 121.9)
- added R25: 1k, MHF:R_0805_2012Metric_Pad1.20x1.40mm_HandSolder, B.Cu at (167.6, 121.9)
- added R26: 1k, MHF:R_0805_2012Metric_Pad1.20x1.40mm_HandSolder, B.Cu at (170.2, 121.9)
- added R27: 1k, MHF:R_0805_2012Metric_Pad1.20x1.40mm_HandSolder, B.Cu at (172.7, 121.9)
- added R28: 1k, MHF:R_0805_2012Metric_Pad1.20x1.40mm_HandSolder, B.Cu at (175.3, 121.9)
- added R29: 1k, MHF:R_0805_2012Metric_Pad1.20x1.40mm_HandSolder, B.Cu at (177.8, 121.9)
- added R3: 1k, MHF:R_0805_2012Metric_Pad1.20x1.40mm_HandSolder, B.Cu at (177.8, 28.0)
- added R30: 1k, MHF:R_0805_2012Metric_Pad1.20x1.40mm_HandSolder, B.Cu at (182.9, 121.9)
- added R31: 1k, MHF:R_0805_2012Metric_Pad1.20x1.40mm_HandSolder, B.Cu at (185.4, 121.9)
- added R32: 1k, MHF:R_0805_2012Metric_Pad1.20x1.40mm_HandSolder, B.Cu at (190.5, 121.9)
- added R33: 1k, MHF:R_0805_2012Metric_Pad1.20x1.40mm_HandSolder, B.Cu at (193.0, 121.9)
- added R34: 1k, MHF:R_0805_2012Metric_Pad1.20x1.40mm_HandSolder, B.Cu at (195.6, 121.9)
- added R35: 1k, MHF:R_0805_2012Metric_Pad1.20x1.40mm_HandSolder, B.Cu at (198.1, 121.9)
- added R36: 5k8, Resistor_SMD:R_0805_2012Metric, B.Cu at (215.9, 43.8)
- added R37: 5k8, Resistor_SMD:R_0805_2012Metric, B.Cu at (213.4, 43.8)
- added R38: 5k8, Resistor_SMD:R_0805_2012Metric, B.Cu at (210.8, 43.8)
- added R39: 5k8, Resistor_SMD:R_0805_2012Metric, B.Cu at (205.7, 43.8)
- added R4: 1k, MHF:R_0805_2012Metric_Pad1.20x1.40mm_HandSolder, B.Cu at (180.3, 28.0)
- added R40: 220, Resistor_SMD:R_0805_2012Metric, B.Cu at (215.9, 47.6)
- added R41: 220, Resistor_SMD:R_0805_2012Metric, B.Cu at (213.4, 47.6)
- added R42: 220, Resistor_SMD:R_0805_2012Metric, B.Cu at (210.8, 47.6)
- added R43: 220, Resistor_SMD:R_0805_2012Metric, B.Cu at (205.7, 47.6)
- added R44: 5k8, Resistor_SMD:R_0805_2012Metric, F.Cu at (215.9, 43.8)
- added R45: 5k8, Resistor_SMD:R_0805_2012Metric, F.Cu at (213.4, 43.8)
- added R46: 5k8, Resistor_SMD:R_0805_2012Metric, F.Cu at (210.8, 43.8)
- added R47: 5k8, Resistor_SMD:R_0805_2012Metric, F.Cu at (205.7, 43.8)
- added R48: 5k8, Resistor_SMD:R_0805_2012Metric, B.Cu at (172.5, 116.0)
- added R49: 5k8, Resistor_SMD:R_0805_2012Metric, B.Cu at (175.1, 116.0)
- added R5: 1k, MHF:R_0805_2012Metric_Pad1.20x1.40mm_HandSolder, B.Cu at (182.9, 28.0)
- added R50: 5k8, Resistor_SMD:R_0805_2012Metric, B.Cu at (177.6, 116.0)
- added R51: 5k8, Resistor_SMD:R_0805_2012Metric, B.Cu at (182.7, 116.0)
- added R52: 220, Resistor_SMD:R_0805_2012Metric, B.Cu at (172.5, 112.2)
- added R53: 220, Resistor_SMD:R_0805_2012Metric, B.Cu at (175.1, 112.2)
- added R54: 220, Resistor_SMD:R_0805_2012Metric, B.Cu at (177.6, 112.2)
- added R55: 220, Resistor_SMD:R_0805_2012Metric, B.Cu at (182.7, 112.2)
- added R56: 5k8, Resistor_SMD:R_0805_2012Metric, F.Cu at (172.5, 116.0)
- added R57: 5k8, Resistor_SMD:R_0805_2012Metric, F.Cu at (175.1, 116.0)
- added R58: 5k8, Resistor_SMD:R_0805_2012Metric, F.Cu at (177.6, 116.0)
- added R59: 5k8, Resistor_SMD:R_0805_2012Metric, F.Cu at (182.7, 116.0)
- added R6: 1k, MHF:R_0805_2012Metric_Pad1.20x1.40mm_HandSolder, B.Cu at (165.1, 27.9)
- added R60: 1M, MHF:R_0805_2012Metric_Pad1.20x1.40mm_HandSolder, F.Cu at (224.7, 120.4)
- added R61: 1k, MHF:R_0805_2012Metric_Pad1.20x1.40mm_HandSolder, F.Cu at (232.0, 29.1)
- added R62: 1k, MHF:R_0805_2012Metric_Pad1.20x1.40mm_HandSolder, B.Cu at (195.3, 84.1)
- added R63: 3k3, MHF:R_0805_2012Metric_Pad1.20x1.40mm_HandSolder, F.Cu at (188.6, 47.0)
- added R64: 10k, MHF:R_0805_2012Metric_Pad1.20x1.40mm_HandSolder, B.Cu at (181.6, 54.6)
- added R65: 1k, MHF:R_0805_2012Metric_Pad1.20x1.40mm_HandSolder, B.Cu at (215.9, 121.9)
- added R66: 1k, MHF:R_0805_2012Metric_Pad1.20x1.40mm_HandSolder, B.Cu at (186.1, 31.8)
- added R7: 1k, MHF:R_0805_2012Metric_Pad1.20x1.40mm_HandSolder, B.Cu at (167.6, 27.9)
- added R8: 1k, MHF:R_0805_2012Metric_Pad1.20x1.40mm_HandSolder, B.Cu at (189.2, 27.9)
- added R9: 1k, MHF:R_0805_2012Metric_Pad1.20x1.40mm_HandSolder, B.Cu at (191.8, 27.9)
- added S1: Reset, MHF:G_Arduino_switch, F.Cu at (191.8, 32.4)
- added TP1: 7, MHF:TestPoint_Pad_1.0x1.0mm, B.Cu at (225.6, 49.3)
- added TP10: 1, MHF:TestPoint_Pad_1.0x1.0mm, B.Cu at (236.7, 60.3)
- added TP11: 2, MHF:TestPoint_Pad_1.0x1.0mm, B.Cu at (236.7, 58.5)
- added TP12: 3, MHF:TestPoint_Pad_1.0x1.0mm, B.Cu at (236.7, 56.8)
- added TP13: 4, MHF:TestPoint_Pad_1.0x1.0mm, B.Cu at (236.7, 54.7)
- added TP14: 5, MHF:TestPoint_Pad_1.0x1.0mm, B.Cu at (236.7, 53.0)
- added TP15: 6, MHF:TestPoint_Pad_1.0x1.0mm, B.Cu at (236.7, 51.2)
- added TP16: 7, MHF:TestPoint_Pad_1.0x1.0mm, B.Cu at (236.7, 49.4)
- added TP17: D, MHF:TestPoint_Pad_1.0x1.0mm, B.Cu at (234.9, 43.4)
- added TP18: Clk, MHF:TestPoint_Pad_1.0x1.0mm, B.Cu at (234.9, 41.7)
- added TP19: Q, MHF:TestPoint_Pad_1.0x1.0mm, B.Cu at (234.9, 38.4)
- added TP2: 0, MHF:TestPoint_Pad_1.0x1.0mm, B.Cu at (225.6, 62.1)
- added TP20: ~{Q}, MHF:TestPoint_Pad_1.0x1.0mm, B.Cu at (234.9, 36.6)
- added TP21: ~{R}, MHF:TestPoint_Pad_1.0x1.0mm, B.Cu at (234.9, 45.0)
- added TP22: ~{S}, MHF:TestPoint_Pad_1.0x1.0mm, B.Cu at (234.9, 39.9)
- added TP23: N3, MHF:TestPoint_Pad_1.0x1.0mm, B.Cu at (225.4, 110.8)
- added TP24: N4, MHF:TestPoint_Pad_1.0x1.0mm, B.Cu at (236.5, 109.5)
- added TP25: N5, MHF:TestPoint_Pad_1.0x1.0mm, B.Cu at (236.5, 113.0)
- added TP26: N6, MHF:TestPoint_Pad_1.0x1.0mm, B.Cu at (236.5, 116.6)
- added TP27: ~{N3}, MHF:TestPoint_Pad_1.0x1.0mm, B.Cu at (225.4, 109.2)
- added TP28: ~{N4}, MHF:TestPoint_Pad_1.0x1.0mm, B.Cu at (236.5, 107.7)
- added TP29: ~{N5}, MHF:TestPoint_Pad_1.0x1.0mm, B.Cu at (236.5, 111.3)
- added TP3: 1, MHF:TestPoint_Pad_1.0x1.0mm, B.Cu at (225.6, 60.3)
- added TP30: ~{N6}, MHF:TestPoint_Pad_1.0x1.0mm, B.Cu at (236.5, 114.8)
- added TP31: IO, MHF:TestPoint_Pad_1.0x1.0mm, B.Cu at (227.3, 101.6)
- added TP32: IO, MHF:TestPoint_Pad_1.0x1.0mm, B.Cu at (229.2, 101.6)
- added TP33: IO, MHF:TestPoint_Pad_1.0x1.0mm, B.Cu at (231.1, 101.6)
- added TP34: IO, MHF:TestPoint_Pad_1.0x1.0mm, B.Cu at (233.0, 101.6)
- added TP35: IO, MHF:TestPoint_Pad_1.0x1.0mm, B.Cu at (234.9, 101.6)
- added TP36: IO, MHF:TestPoint_Pad_1.0x1.0mm, B.Cu at (234.9, 105.4)
- added TP37: IO, MHF:TestPoint_Pad_1.0x1.0mm, B.Cu at (233.0, 105.4)
- added TP38: IO, MHF:TestPoint_Pad_1.0x1.0mm, B.Cu at (228.0, 68.6)
- added TP39: IO, MHF:TestPoint_Pad_1.0x1.0mm, B.Cu at (229.9, 68.6)
- added TP4: 2, MHF:TestPoint_Pad_1.0x1.0mm, B.Cu at (225.6, 58.5)
- added TP40: IO, MHF:TestPoint_Pad_1.0x1.0mm, B.Cu at (231.8, 68.6)
- added TP41: IO, MHF:TestPoint_Pad_1.0x1.0mm, B.Cu at (233.7, 68.6)
- added TP42: IO, MHF:TestPoint_Pad_1.0x1.0mm, B.Cu at (235.6, 68.6)
- added TP43: IO, MHF:TestPoint_Pad_1.0x1.0mm, B.Cu at (228.0, 71.1)
- added TP44: IO, MHF:TestPoint_Pad_1.0x1.0mm, B.Cu at (229.9, 71.1)
- added TP45: IO, MHF:TestPoint_Pad_1.0x1.0mm, B.Cu at (231.8, 71.1)
- added TP46: IO, MHF:TestPoint_Pad_1.0x1.0mm, B.Cu at (233.7, 71.1)
- added TP47: IO, MHF:TestPoint_Pad_1.0x1.0mm, B.Cu at (235.6, 71.1)
- added TP48: IO, MHF:TestPoint_Pad_1.0x1.0mm, B.Cu at (228.0, 74.3)
- added TP49: IO, MHF:TestPoint_Pad_1.0x1.0mm, B.Cu at (229.9, 74.3)
- added TP5: 3, MHF:TestPoint_Pad_1.0x1.0mm, B.Cu at (225.6, 56.8)
- added TP50: IO, MHF:TestPoint_Pad_1.0x1.0mm, B.Cu at (231.8, 74.3)
- added TP51: IO, MHF:TestPoint_Pad_1.0x1.0mm, B.Cu at (233.7, 74.3)
- added TP52: IO, MHF:TestPoint_Pad_1.0x1.0mm, B.Cu at (235.6, 74.3)
- added TP53: IO, MHF:TestPoint_Pad_1.0x1.0mm, B.Cu at (228.0, 79.3)
- added TP54: IO, MHF:TestPoint_Pad_1.0x1.0mm, B.Cu at (229.9, 79.3)
- added TP55: IO, MHF:TestPoint_Pad_1.0x1.0mm, B.Cu at (231.8, 79.3)
- added TP56: IO, MHF:TestPoint_Pad_1.0x1.0mm, B.Cu at (233.7, 79.3)
- added TP57: IO, MHF:TestPoint_Pad_1.0x1.0mm, B.Cu at (235.6, 79.3)
- added TP58: IO, MHF:TestPoint_Pad_1.0x1.0mm, B.Cu at (226.1, 81.8)
- added TP59: IO, MHF:TestPoint_Pad_1.0x1.0mm, B.Cu at (228.0, 81.8)
- added TP6: 4, MHF:TestPoint_Pad_1.0x1.0mm, B.Cu at (225.6, 54.6)
- added TP60: IO, MHF:TestPoint_Pad_1.0x1.0mm, B.Cu at (229.9, 81.8)
- added TP61: IO, MHF:TestPoint_Pad_1.0x1.0mm, B.Cu at (231.8, 81.8)
- added TP62: IO, MHF:TestPoint_Pad_1.0x1.0mm, B.Cu at (233.7, 81.8)
- added TP63: IO, MHF:TestPoint_Pad_1.0x1.0mm, B.Cu at (235.6, 81.8)
- added TP65: I, MHF:TestPoint_Pad_1.0x1.0mm, B.Cu at (228.0, 64.2)
- added TP66: I, MHF:TestPoint_Pad_1.0x1.0mm, B.Cu at (229.9, 64.2)
- added TP67: I, MHF:TestPoint_Pad_1.0x1.0mm, B.Cu at (231.8, 64.2)
- added TP68: I, MHF:TestPoint_Pad_1.0x1.0mm, B.Cu at (233.7, 64.2)
- added TP69: I, MHF:TestPoint_Pad_1.0x1.0mm, B.Cu at (235.6, 64.2)
- added TP7: 5, MHF:TestPoint_Pad_1.0x1.0mm, B.Cu at (225.6, 52.8)
- added TP70: I, MHF:TestPoint_Pad_1.0x1.0mm, B.Cu at (227.3, 98.4)
- added TP71: I, MHF:TestPoint_Pad_1.0x1.0mm, B.Cu at (229.2, 98.4)
- added TP72: I, MHF:TestPoint_Pad_1.0x1.0mm, B.Cu at (231.1, 98.4)
- added TP73: I, MHF:TestPoint_Pad_1.0x1.0mm, B.Cu at (233.0, 98.4)
- added TP74: I, MHF:TestPoint_Pad_1.0x1.0mm, B.Cu at (234.9, 98.4)
- added TP8: 6, MHF:TestPoint_Pad_1.0x1.0mm, B.Cu at (225.6, 51.1)
- added TP9: 0, MHF:TestPoint_Pad_1.0x1.0mm, B.Cu at (236.7, 62.1)
- added ToDo1: J, MHF:PinHeader_1x09_P2.54mm_Vertical, F.Cu at (221.0, 78.7)
- added U10: 74HC14, MHF:SOIC-14_3.9x8.7mm_P1.27mm, B.Cu at (195.6, 114.3)
- added U11: 74HC14, MHF:SOIC-14_3.9x8.7mm_P1.27mm, B.Cu at (208.3, 116.8)
- added U12: 74HC04, MHF:SOIC-14_3.9x8.7mm_P1.27mm, B.Cu at (231.1, 111.8)
- added U13: 74HC74, MHF:SOIC-14_3.9x8.7mm_P1.27mm, B.Cu at (229.6, 40.9)
- added U3: ATF1504AS-10AU100, Gilhad_footprints:ATF1504-AS_TQFP100_long, F.Cu at (203.9, 97.6)
- added U4: MC68B50, Package_DIP:DIP-24_W15.24mm, F.Cu at (238.8, 116.8)
- added U5: 6822, Package_DIP:DIP-40_W15.24mm, F.Cu at (238.8, 83.8)
- added U6: 74HC14, MHF:SOIC-14_3.9x8.7mm_P1.27mm, B.Cu at (175.3, 38.1)
- added U7: 74HC14, MHF:SOIC-14_3.9x8.7mm_P1.27mm, B.Cu at (185.4, 38.1)
- added U8: 74HC14, MHF:SOIC-14_3.9x8.7mm_P1.27mm, B.Cu at (203.2, 35.6)
- added U9: 74HC14, MHF:SOIC-14_3.9x8.7mm_P1.27mm, B.Cu at (213.4, 35.6)
- added Y1: 1.8432 MHz, Gilhad_footprints:Crystal_THT_15_5mm, F.Cu at (218.6, 101.1)
- M3: moved to B.Cu
- moved Cx1 167.3 mm to (261.1, 73.3)
- moved Cx2 167.3 mm to (261.1, 76.9)
- moved Cx3 167.3 mm to (261.1, 80.4)
- moved Cx4 167.3 mm to (261.1, 84.0)
- moved Cx5 167.3 mm to (261.1, 87.5)
- moved Cx6 148.0 mm to (241.5, 88.8), turned to 90 degrees
- moved Cx15 139.1 mm to (245.3, 88.4), turned to 90 degrees
- moved J43 136.9 mm to (266.1, 99.6)
- moved J46 136.9 mm to (266.1, 104.7)
- moved J47 136.9 mm to (266.1, 107.3)
- moved J48 136.9 mm to (266.1, 109.8)
- moved J49 136.9 mm to (266.1, 112.3)
- moved J50 136.9 mm to (266.1, 114.9)
- moved J53 136.9 mm to (266.1, 102.2)
- moved J59 136.9 mm to (266.1, 97.1)
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Connections:
- net /A_16 renamed /mA_16
- net /B_16 renamed /mB_16
- net A_HALT renamed /mA_HALT
- net A_READ renamed /mA_READ
- net A_SHARE_DIRTY renamed /mA_SHARE_DIRTY
- net A_SHARE_GRANTED renamed /mA_SHARE_GRANTED
- net A_SHARE_REQUEST renamed /mA_SHARE_REQUEST
- net A_SHARE_SELECT renamed /mA_SHARE_SELECT
- net B_HALT renamed /mB_HALT
- net B_READ renamed /mB_READ
- net B_SHARE_DIRTY renamed /mB_SHARE_DIRTY
- net B_SHARE_GRANTED renamed /mB_SHARE_GRANTED
- net B_SHARE_REQUEST renamed /mB_SHARE_REQUEST
- net B_SHARE_SELECT renamed /mB_SHARE_SELECT
- J4 pad 11: A0 -> /CA0
- J4 pad 12: A1 -> /CA1
- J4 pad 13: A2 -> /CA2
- J4 pad 14: A3 -> /CA3
- J4 pad 15: A4 -> /CA4
- J4 pad 16: A5 -> /CA5
- J4 pad 17: A6 -> /CA6
- J4 pad 18: A7 -> /CA7
- J4 pad 19: A8 -> /CA8
- J4 pad 20: A9 -> /CA9
- J4 pad 21: A10 -> /CA10
- J4 pad 22: A11 -> /CA11
- J4 pad 23: A12 -> /A12
- J4 pad 24: A13 -> /A13
- J4 pad 25: A14 -> /A14
- J4 pad 26: A15 -> /A15
- J4 pad 53: unconnected-(J4-Pin_53-Pad53) -> /~{Write}
- J4 pad 54: unconnected-(J4-Pin_54-Pad54) -> /~{Read}
- J4 pad 55: unconnected-(J4-Pin_55-Pad55) -> /~{NMI}
- J4 pad 56: unconnected-(J4-Pin_56-Pad56) -> /~{IRQ}
- J4 pad 57: unconnected-(J4-Pin_57-Pad57) -> /~{FIRQ}
- J4 pad 58: unconnected-(J4-Pin_58-Pad58) -> /~{Dev_Sel_3}
- J4 pad 59: unconnected-(J4-Pin_59-Pad59) -> /~{Dev_Sel_4}
- J4 pad 60: unconnected-(J4-Pin_60-Pad60) -> /~{Dev_Sel_5}
- J4 pad 61: unconnected-(J4-Pin_61-Pad61) -> /E
- J6 pad 11: A0 -> /CA0
- J6 pad 12: A1 -> /CA1
- J6 pad 13: A2 -> /CA2
- J6 pad 14: A3 -> /CA3
- J6 pad 15: A4 -> /CA4
- J6 pad 16: A5 -> /CA5
- J6 pad 17: A6 -> /CA6
- J6 pad 18: A7 -> /CA7
- J6 pad 19: A8 -> /CA8
- J6 pad 20: A9 -> /CA9
- J6 pad 21: A10 -> /CA10
- J6 pad 22: A11 -> /CA11
- J6 pad 23: A12 -> /A12
- J6 pad 24: A13 -> /A13
- J6 pad 25: A14 -> /A14
- J6 pad 26: A15 -> /A15
- J6 pad 53: unconnected-(J6-Pin_53-Pad53) -> /~{Write}
- J6 pad 54: unconnected-(J6-Pin_54-Pad54) -> /~{Read}
- J6 pad 55: unconnected-(J6-Pin_55-Pad55) -> /~{NMI}
- J6 pad 56: unconnected-(J6-Pin_56-Pad56) -> /~{IRQ}
- J6 pad 57: unconnected-(J6-Pin_57-Pad57) -> /~{FIRQ}
- J6 pad 58: unconnected-(J6-Pin_58-Pad58) -> /~{Dev_Sel_3}
- J6 pad 59: unconnected-(J6-Pin_59-Pad59) -> /~{Dev_Sel_4}
- J6 pad 60: unconnected-(J6-Pin_60-Pad60) -> /~{Dev_Sel_5}
- J6 pad 61: unconnected-(J6-Pin_61-Pad61) -> /E
- M3 pad 1: A11 -> /CA11
- M3 pad 10: unconnected-(M3-A16-Pad10) -> GA16
- M3 pad 11: unconnected-(M3-A14-Pad11) -> /A14
- M3 pad 12: unconnected-(M3-A12-Pad12) -> /A12
- M3 pad 13: A7 -> /CA7
- M3 pad 14: A6 -> /CA6
- M3 pad 15: A5 -> /CA5
- M3 pad 16: A4 -> /CA4
- M3 pad 17: A3 -> /CA3
- M3 pad 18: A2 -> /CA2
- M3 pad 19: A1 -> /CA1
- M3 pad 2: A9 -> /CA9
- M3 pad 20: A0 -> /CA0
- M3 pad 24: unconnected-(M3-GND-Pad24) -> GND
- M3 pad 3: A8 -> /CA8
- M3 pad 30: unconnected-(M3-~{CS1}/~{CE1}-Pad30) -> ~{Dev_Sel_0}
- M3 pad 31: A10 -> /CA10
- M3 pad 32: unconnected-(M3-~{OE}-Pad32) -> /~{Read}
- M3 pad 4: unconnected-(M3-A13-Pad4) -> /A13
- M3 pad 5: unconnected-(M3-~{WE}-Pad5) -> /~{Write}
- M3 pad 6: unconnected-(M3-CS2/CE2-Pad6) -> +5V
- M3 pad 7: unconnected-(M3-A15-Pad7) -> /A15
- M3 pad 8: unconnected-(M3-VCC-Pad8) -> +5V
- U1 pad 1: unconnected-(U1-VSS-Pad1) -> GND
- U1 pad 10: A2 -> /CA2
- U1 pad 11: A3 -> /CA3
- U1 pad 12: A4 -> /CA4
- U1 pad 13: A5 -> /CA5
- U1 pad 14: A6 -> /CA6
- U1 pad 15: A7 -> /CA7
- U1 pad 16: A8 -> /CA8
- U1 pad 17: A9 -> /CA9
- U1 pad 18: A10 -> /CA10
- U1 pad 19: A11 -> /CA11
- U1 pad 2: unconnected-(U1-~{NMI}-Pad2) -> /~{NMI}
- U1 pad 20: A12 -> CA12
- U1 pad 21: A13 -> CA13
- U1 pad 22: A14 -> CA14
- U1 pad 23: A15 -> CA15
- U1 pad 3: unconnected-(U1-~{IRQ}-Pad3) -> /~{IRQ}
- U1 pad 32: unconnected-(U1-R/~{W}-Pad32) -> R~{W}
- U1 pad 33: unconnected-(U1-~{DMA/BREQ}-Pad33) -> ~{DMA/BREQ}
- U1 pad 34: unconnected-(U1-E-Pad34) -> /E
- U1 pad 35: unconnected-(U1-Q-Pad35) -> Q
- U1 pad 36: unconnected-(U1-MRDY-Pad36) -> MRDY
- U1 pad 37: unconnected-(U1-~{RESET}-Pad37) -> MasterReset
- U1 pad 4: unconnected-(U1-~{FIRQ}-Pad4) -> /~{FIRQ}
- U1 pad 40: unconnected-(U1-~{HALT}-Pad40) -> ~{HALT}
- U1 pad 5: unconnected-(U1-BS-Pad5) -> BS
- U1 pad 6: unconnected-(U1-BA-Pad6) -> BA
- U1 pad 8: A0 -> /CA0
- U1 pad 9: A1 -> /CA1
- U2 pad 10: unconnected-(U2-I/O-Pad10) -> /CA3
- U2 pad 100: unconnected-(U2-I/O-Pad100) -> MR0
- U2 pad 12: unconnected-(U2-I/O/PD1-Pad12) -> /CA4
- U2 pad 13: unconnected-(U2-I/O-Pad13) -> /CA5
- U2 pad 14: unconnected-(U2-I/O-Pad14) -> /CA6
- U2 pad 16: unconnected-(U2-I/O-Pad16) -> /CA7
- U2 pad 17: unconnected-(U2-I/O-Pad17) -> /CA8
- U2 pad 19: unconnected-(U2-I/O-Pad19) -> /CA9
- U2 pad 20: unconnected-(U2-I/O-Pad20) -> /CA10
- U2 pad 21: unconnected-(U2-I/O-Pad21) -> /CA11
- U2 pad 23: unconnected-(U2-I/O-Pad23) -> CA12
- U2 pad 25: unconnected-(U2-I/O-Pad25) -> CA13
- U2 pad 29: unconnected-(U2-I/O-Pad29) -> CA14
- U2 pad 30: unconnected-(U2-I/O-Pad30) -> CA15
- U2 pad 31: unconnected-(U2-I/O-Pad31) -> /E
- U2 pad 32: unconnected-(U2-I/O-Pad32) -> R~{W}
- U2 pad 33: unconnected-(U2-I/O-Pad33) -> MasterReset
- U2 pad 35: unconnected-(U2-I/O-Pad35) -> Net-(TP63-Pad1)
- U2 pad 36: unconnected-(U2-I/O-Pad36) -> Net-(TP62-Pad1)
- U2 pad 37: unconnected-(U2-I/O-Pad37) -> Net-(TP61-Pad1)
- U2 pad 40: unconnected-(U2-I/O-Pad40) -> Net-(TP60-Pad1)
- U2 pad 41: unconnected-(U2-I/O-Pad41) -> Net-(TP59-Pad1)
- U2 pad 42: unconnected-(U2-I/O/PD2-Pad42) -> Net-(U2-I/O/PD2)
- U2 pad 44: unconnected-(U2-I/O-Pad44) -> Net-(TP57-Pad1)
- U2 pad 45: unconnected-(U2-I/O-Pad45) -> Net-(TP56-Pad1)
- U2 pad 46: unconnected-(U2-I/O-Pad46) -> Net-(TP55-Pad1)
- U2 pad 47: unconnected-(U2-I/O-Pad47) -> Net-(TP54-Pad1)
- U2 pad 48: unconnected-(U2-I/O-Pad48) -> Net-(TP53-Pad1)
- U2 pad 52: unconnected-(U2-I/O-Pad52) -> Net-(TP52-Pad1)
- U2 pad 54: unconnected-(U2-I/O-Pad54) -> Net-(TP51-Pad1)
- U2 pad 56: unconnected-(U2-I/O-Pad56) -> Net-(TP50-Pad1)
- U2 pad 57: unconnected-(U2-I/O-Pad57) -> Net-(TP49-Pad1)
- U2 pad 58: unconnected-(U2-I/O-Pad58) -> Net-(TP48-Pad1)
- U2 pad 6: unconnected-(U2-I/O-Pad6) -> /CA0
- U2 pad 60: unconnected-(U2-I/O-Pad60) -> Net-(TP47-Pad1)
- U2 pad 61: unconnected-(U2-I/O-Pad61) -> Net-(TP46-Pad1)
- U2 pad 63: unconnected-(U2-I/O-Pad63) -> Net-(TP45-Pad1)
- U2 pad 64: unconnected-(U2-I/O-Pad64) -> Net-(TP44-Pad1)
- U2 pad 65: unconnected-(U2-I/O-Pad65) -> Net-(TP43-Pad1)
- U2 pad 67: unconnected-(U2-I/O-Pad67) -> Net-(TP42-Pad1)
- U2 pad 68: unconnected-(U2-I/O-Pad68) -> Net-(TP41-Pad1)
- U2 pad 69: unconnected-(U2-I/O-Pad69) -> Net-(TP40-Pad1)
- U2 pad 71: unconnected-(U2-I/O-Pad71) -> Net-(TP39-Pad1)
- U2 pad 75: unconnected-(U2-I/O-Pad75) -> Net-(TP38-Pad1)
- U2 pad 76: unconnected-(U2-I/O-Pad76) -> ~{Dev_Sel_7}
- U2 pad 79: unconnected-(U2-I/O-Pad79) -> ~{Dev_Sel_6}
- U2 pad 8: unconnected-(U2-I/O-Pad8) -> /CA1
- U2 pad 80: unconnected-(U2-I/O-Pad80) -> /~{Dev_Sel_5}
- U2 pad 81: unconnected-(U2-I/O-Pad81) -> /~{Dev_Sel_4}
- U2 pad 83: unconnected-(U2-I/O-Pad83) -> /~{Dev_Sel_3}
- U2 pad 84: unconnected-(U2-I/O-Pad84) -> ~{Dev_Sel_2}
- U2 pad 85: unconnected-(U2-I/O/GCLK3-Pad85) -> Net-(U2-I/O/GCLK3)
- U2 pad 87: unconnected-(U2-INPUT/GCLK1-Pad87) -> Net-(U2-INPUT/GCLK1)
- U2 pad 88: unconnected-(U2-12V/INPUT/OE1-Pad88) -> Net-(U2-12V/INPUT/OE1)
- U2 pad 89: unconnected-(U2-INPUT/GCLR-Pad89) -> Net-(U2-INPUT/GCLR)
- U2 pad 9: unconnected-(U2-I/O-Pad9) -> /CA2
- U2 pad 90: unconnected-(U2-INPUT/OE2/GCLK2-Pad90) -> Net-(U2-INPUT/OE2/GCLK2)
- U2 pad 92: unconnected-(U2-I/O-Pad92) -> ~{Dev_Sel_1}
- U2 pad 93: unconnected-(U2-I/O-Pad93) -> ~{Dev_Sel_0}
- U2 pad 94: unconnected-(U2-I/O-Pad94) -> /~{Write}
- U2 pad 96: unconnected-(U2-I/O-Pad96) -> /~{Read}
- U2 pad 97: unconnected-(U2-I/O-Pad97) -> MR3
- U2 pad 98: unconnected-(U2-I/O-Pad98) -> MR2
- U2 pad 99: unconnected-(U2-I/O-Pad99) -> MR1
Routing:
- net MasterReset: track 6.54 -> 0.00 mm
- net A13: track 6.22 -> 0.00 mm
- net /mB_READ: track 6.21 -> 0.00 mm
- net /mB_SHARE_SELECT: track 6.15 -> 0.00 mm
- net /mA_SHARE_SELECT: track 6.07 -> 0.00 mm
- net A_S_WRITE: track 6.06 -> 0.00 mm
- net /mA_16: track 5.96 -> 0.00 mm
- net B_G_A_DIR: track 5.93 -> 0.00 mm
- net B_S_SELECT: track 5.91 -> 0.00 mm
- net A14: track 5.91 -> 0.00 mm
- net /mA_HALT: track 5.91 -> 0.00 mm
- net D5: track 5.91 -> 0.00 mm
- net D2: track 5.91 -> 0.00 mm
- net A10: track 5.91 -> 0.00 mm
- net D6: track 5.91 -> 0.00 mm
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