File: HW/KiCad/retro-002/retro-002.kicad_sch (KiCad schematic)
At the start: 322 parts, among them J1 Conn_02x05_JTAG, J100 x, J101 x, J102 x, J103 x, J104 x, J105 x, J106 x, J12 Reset, J2 Conn_02x05_JTAG, J21 x, J22 x, J3 Serial, J37 x, J38 x, J39 x, J4 SysBus, J40 x, J41 x, J42 x, J43 x, J44 x, J45 x, J46 x, J47 x, J48 x, J49 x, J50 x, J51 x, J52 x, J53 x, J54 x, J55 x, J56 x, J57 x, J58 x, J59 x, J6 SysBus, J60 x, J61 x, J62 x, J63 x, J64 x, J65 x, J66 x, J67 x, J68 x, J69 x, J7 Conn_01x16_Pin, J70 x, J71 x, J72 x, J73 x, J74 x, J75 x, J76 x, J77 x, J78 x, J79 x, J80 x, J81 x, J82 x, J83 x, J84 x, J85 x, J86 x, J87 x, J88 x, J89 x, J90 x, J91 x, J92 x, J93 x, J94 x, J95 x, J96 x, J97 x, J98 x, J99 x, M3 CY7C109D-10ZXI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

Commit message: retro-002, mozna funkcni?
Parts:
- removed Cx1, Cx2, Cx3, Cx4, Cx5: Cx, MHF:C_Disc_D3.0mm_W2.0mm_P2.50mm, symbol MHF:C
- removed TP31, TP32, TP33, TP34, TP35, TP36, TP37, TP56, TP57, TP58, TP59, TP60, TP61, TP62, TP63: IO, MHF:TestPoint_Pad_1.0x1.0mm, symbol MHF:TestPoint_Probe
- added L36, L37, L38, L39, L40, L41, L42, L43, L44, L45, L46, L47, L48, L49, L50, L51, L52, L53, L54, L55, L56, L57, L58, L59: A0, MHF:LED_0805_2012Metric, symbol MHF:LED
- added R67, R68: 4k8, MHF:R_0805_2012Metric_Pad1.20x1.40mm_HandSolder, symbol MHF:R
- added R69, R70, R71, R72, R73, R74, R75, R76, R77, R78, R79, R80, R81, R82, R83, R84, R85, R86, R87, R88, R89, R90, R91, R92: 1k, MHF:R_0805_2012Metric_Pad1.20x1.40mm_HandSolder, symbol MHF:R
Connections:
- net ~{Dev_Write} is gone; now on net Dev_E: J4.53 (Pin_53), J6.53 (Pin_53)
- net +5V: now also R67.1, R68.1
- net BA: now also U2.36 (I/O), U3.83 (I/O)
- net BS: now also U2.45 (I/O), U3.71 (I/O)
- net Dev_E: no longer J4.61 (Pin_61), J6.61 (Pin_61)
- net GND: now also L36.1 (K), L37.1 (K), L38.1 (K), L39.1 (K), L40.1 (K), L41.1 (K), L42.1 (K), L43.1 (K), L44.1 (K), L45.1 (K), L46.1 (K), L47.1 (K), L48.1 (K), L49.1 (K), L50.1 (K), L51.1 (K), L52.1 (K), L53.1 (K), L54.1 (K), L55.1 (K), L56.1 (K), L57.1 (K), L58.1 (K), L59.1 (K)
- net MRDY: now also U2.44 (I/O), U3.75 (I/O)
- net Rx: now also R91.2
- net Tx: now also R92.2
- net mA_SHARE_DIRTY: now also R67.2
- net mB_SHARE_DIRTY: now also R68.2
- net vCA1: now also R90.2
- net vCA2: now also R89.2
- net vCB1: now also R88.2
- net vCB2: now also R87.2
- net v~{IRQA}: now also R86.2
- net v~{IRQB}: now also R85.2
- net ~{DMA/BREQ}: now also U2.42 (I/O/PD2), U3.76 (I/O)
- net ~{FIRQ}: now also U2.41 (I/O), U3.79 (I/O)
- net ~{HALT}: now also U2.35 (I/O)
- net ~{IRQ}: now also U2.40 (I/O), U3.80 (I/O)
- net ~{NMI}: now also U2.37 (I/O), U3.81 (I/O)
- net at PB1.1 (Pin_1), U5.10 (PB0): now also R77.2
- net at PB1.2 (Pin_2), U5.11 (PB1): now also R78.2
- net at PB1.3 (Pin_3), U5.12 (PB2): now also R79.2
- net at PB1.4 (Pin_4), U5.13 (PB3): now also R80.2
- net at PB1.5 (Pin_5), U5.14 (PB4): now also R81.2
- net at PB1.6 (Pin_6), U5.15 (PB5): now also R82.2
- net at PB1.7 (Pin_7), U5.16 (PB6): now also R83.2
- net at PB1.8 (Pin_8), R61.1, U5.17 (PB7): now also R84.2
- net at PA1.1 (Pin_1), U5.2 (PA0): now also R69.2
- net at PA1.2 (Pin_2), U5.3 (PA1): now also R70.2
- net at PA1.3 (Pin_3), U5.4 (PA2): now also R71.2
- net at PA1.4 (Pin_4), U5.5 (PA3): now also R72.2
- net at PA1.5 (Pin_5), U5.6 (PA4): now also R73.2
- net at PA1.6 (Pin_6), U5.7 (PA5): now also R74.2
- net at PA1.7 (Pin_7), U5.8 (PA6): now also R75.2
- net at PA1.8 (Pin_8), U5.9 (PA7): now also R76.2
- net ~{Dev_Read} renamed Dev_R~{W}
- new net: L57.2 (A), R90.1
- new net: L39.2 (A), R72.1
- new net: L50.2 (A), R83.1
- new net: L36.2 (A), R69.1
- new net: L45.2 (A), R78.1
- new net: L46.2 (A), R79.1
- new net: L53.2 (A), R86.1
- new net: L37.2 (A), R70.1
- new net: L58.2 (A), R91.1
- new net: L48.2 (A), R81.1
- new net: L47.2 (A), R80.1
- new net: L59.2 (A), R92.1
- new net: L42.2 (A), R75.1
- new net: L49.2 (A), R82.1
- new net: L40.2 (A), R73.1
- new net: L43.2 (A), R76.1
- new net: L54.2 (A), R87.1
- new net: L44.2 (A), R77.1
- new net: L38.2 (A), R71.1
- new net: L52.2 (A), R85.1
- new net: L56.2 (A), R89.1
- new net: L55.2 (A), R88.1
- new net: L41.2 (A), R74.1
- new net: L51.2 (A), R84.1
- new net ~{Dev_4}: J4.61 (Pin_61), J6.61 (Pin_61)
Other:
- note added: "5 E, R/~W ~Reset, HALT, BA"
- note added: "5 E, R/~W ~Reset, ~HALT, BA"
- note added: "6"
- note added: "For future use maybe"
- note added: "I2C style pullup"
- note added: "~Reset, NMI, IRQ, FIRQ,E,R~{W}"
- note removed: "3 E, R/~W ~Reset"
- note removed: "4 E, R/~W ~Reset, ~HALT"
- note removed: "~Reset, NMI, IRQ, FIRQ"
- note removed: "~Reset, NMI, IRQ, FIRQ,E"
- moved on the sheet: Jx4, LS1, PB1, Q1, U13A
