File: HW/KiCad/retro-002/retro-002.kicad_sch (KiCad schematic)
At the start: 352 parts, among them J1 Conn_02x05_JTAG, J100 x, J101 x, J102 x, J103 x, J104 x, J105 x, J106 x, J12 Reset, J2 Conn_02x05_JTAG, J21 x, J22 x, J3 Serial, J37 x, J38 x, J39 x, J4 SysBus, J40 x, J41 x, J42 x, J43 x, J44 x, J45 x, J46 x, J47 x, J48 x, J49 x, J50 x, J51 x, J52 x, J53 x, J54 x, J55 x, J56 x, J57 x, J58 x, J59 x, J6 SysBus, J60 x, J61 x, J62 x, J63 x, J64 x, J65 x, J66 x, J67 x, J68 x, J69 x, J7 Conn_01x16_Pin, J70 x, J71 x, J72 x, J73 x, J74 x, J75 x, J76 x, J77 x, J78 x, J79 x, J80 x, J81 x, J82 x, J83 x, J84 x, J85 x, J86 x, J87 x, J88 x, J89 x, J90 x, J91 x, J92 x, J93 x, J94 x, J95 x, J96 x, J97 x, J98 x, J99 x, M3 CY7C109D-10ZXI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

Commit message: Pridana EEPROM, ucesano, pridana rozpracovana PLD
Parts:
- removed TP38, TP39, TP40, TP41, TP42, TP43, TP44, TP45, TP46, TP47, TP48: IO, MHF:TestPoint_Pad_1.0x1.0mm, symbol MHF:TestPoint_Probe
- removed TP66, TP68, TP69, TP71, TP73, TP74: I, MHF:TestPoint_Pad_1.0x1.0mm, symbol MHF:TestPoint_Probe
- removed ToDo1: J, MHF:PinHeader_1x09_P2.54mm_Vertical, symbol MHF:Conn_01x09
- added J5, J8: x, MHF:PinHole_1x01_2.54xrectangle, symbol MHF:Conn_01x01
- added Jx2: BootFrom, MHF:PinHeader_1x03_P2.54mm_Vertical, symbol MHF:Conn_01x03
- added R93, R94: 50k, MHF:R_0805_2012Metric_Pad1.20x1.40mm_HandSolder, symbol MHF:R
- added R95, R96: 10k, MHF:R_0805_2012Metric_Pad1.20x1.40mm_HandSolder, symbol MHF:R
- added R97: 1k, MHF:R_0805_2012Metric_Pad1.20x1.40mm_HandSolder, symbol MHF:R
- added RomMapped1: RomMapped, MHF:LED_0805_2012Metric, symbol MHF:LED
- added TP31: DEV7, MHF:TestPoint_Pad_1.0x1.0mm, symbol MHF:TestPoint_Probe
- added TP32: DMA, MHF:TestPoint_Pad_1.0x1.0mm, symbol MHF:TestPoint_Probe
- added TP33: MRDY, MHF:TestPoint_Pad_1.0x1.0mm, symbol MHF:TestPoint_Probe
- added TP34: BA, MHF:TestPoint_Pad_1.0x1.0mm, symbol MHF:TestPoint_Probe
- added TP35: BS, MHF:TestPoint_Pad_1.0x1.0mm, symbol MHF:TestPoint_Probe
- added TP36: Q, MHF:TestPoint_Pad_1.0x1.0mm, symbol MHF:TestPoint_Probe
- added TP56, TP57, TP58: IO, MHF:TestPoint_Pad_1.0x1.0mm, symbol MHF:TestPoint_Probe
- added U14: 28C256, Package_DIP:DIP-28_W15.24mm, symbol Memory_EEPROM:28C256
- U4: footprint Package_DIP:DIP-24_W15.24mm -> Gilhad_footprints:DIP-24_W15.24mm
- U5: footprint Package_DIP:DIP-40_W15.24mm -> Gilhad_footprints:DIP-40_W15.24mm
Connections:
- net +5V: now also J5.1 (Pin_1), R93.1, R94.1, R95.2, U14.28 (VCC)
- net BA: now also U2.33 (I/O), TP34.1; no longer U2.36 (I/O)
- net BS: now also U2.42 (I/O/PD2), TP35.1; no longer U2.45 (I/O)
- net CA0: now also U14.10 (A0)
- net CA1: now also U14.9 (A1)
- net CA10: now also U14.21 (A10)
- net CA11: now also U14.23 (A11)
- net CA12: now also U3.20 (I/O); no longer U3.23 (I/O)
- net CA13: now also U3.21 (I/O); no longer U3.25 (I/O)
- net CA14: now also U3.23 (I/O); no longer U3.29 (I/O)
- net CA15: now also U3.25 (I/O); no longer U3.30 (I/O)
- net CA2: now also U14.8 (A2)
- net CA3: now also U14.7 (A3)
- net CA4: now also U14.6 (A4)
- net CA5: now also U14.5 (A5)
- net CA6: now also U14.4 (A6)
- net CA7: now also U14.3 (A7)
- net CA8: now also U14.25 (A8)
- net CA9: now also U14.24 (A9)
- net D0: now also U2.58 (I/O), U14.11 (D0)
- net D1: now also U2.60 (I/O), U14.12 (D1)
- net D2: now also U2.61 (I/O), U14.13 (D2)
- net D3: now also U2.63 (I/O), U14.15 (D3)
- net D4: now also U2.64 (I/O), U14.16 (D4)
- net D5: now also U2.65 (I/O), U14.17 (D5)
- net D6: now also U2.67 (I/O), U14.18 (D6)
- net D7: now also U2.68 (I/O), U14.19 (D7)
- net E: now also U2.87 (INPUT/GCLK1), U3.87 (INPUT/GCLK1); no longer U2.31 (I/O), U3.17 (I/O)
- net GA12: now also U14.2 (A12)
- net GA13: now also U14.26 (A13)
- net GA14: now also U14.1 (A14)
- net GND: now also J8.1 (Pin_1), R96.2, RomMapped1.1 (K), U14.14 (GND)
- net MRDY: now also U2.41 (I/O), TP33.1; no longer U2.44 (I/O)
- net Q: now also U2.90 (INPUT/OE2/GCLK2), U3.90 (INPUT/OE2/GCLK2), TP36.1
- net R~{W}: now also U2.31 (I/O), U3.17 (I/O); no longer U2.32 (I/O), U3.19 (I/O)
- net mA_HALT: now also R93.2
- net mB_HALT: now also R94.2
- net ~{DMA/BREQ}: now also U2.40 (I/O), TP32.1; no longer U2.42 (I/O/PD2)
- net ~{Dev_Sel_7}: now also TP31.1
- net ~{FIRQ}: now also U2.37 (I/O); no longer U2.41 (I/O)
- net ~{HALT}: now also U2.32 (I/O), U3.19 (I/O); no longer U2.35 (I/O), U3.21 (I/O)
- net ~{IRQ}: now also U2.36 (I/O); no longer U2.40 (I/O)
- net ~{NMI}: now also U2.35 (I/O); no longer U2.37 (I/O)
- net ~{RESET}: now also U2.89 (INPUT/GCLR), U3.89 (INPUT/GCLR); no longer U2.33 (I/O), U3.20 (I/O)
- net ~{Read}: now also U14.22 (~{OE})
- net ~{Write}: now also U14.27 (~{WE})
- net at U3.85 (I/O/GCLK3): now also TP70.1
- net at TP55.1: now also U2.44 (I/O); no longer U2.46 (I/O)
- net at U2.47 (I/O): now also TP56.1; no longer TP54.1
- net at U2.48 (I/O): now also TP57.1; no longer TP53.1
- net at U2.52 (I/O): now also TP49.1; no longer TP52.1
- net at U2.54 (I/O): now also TP50.1; no longer TP51.1
- net at U2.56 (I/O): now also TP51.1; no longer TP50.1
- net at U2.57 (I/O): now also TP52.1; no longer TP49.1
- net RomMapped: now reaches U2.69 (I/O)
- net RomMapped: now also R97.2
- net BootSrc: now reaches U2.71 (I/O)
- net BootSrc: now also Jx2.2 (Pin_2)
- net ~{ROM}: now reaches U2.75 (I/O)
- net ~{ROM}: now also U3.30 (I/O), U14.20 (~{CS})
- net at U2.85 (I/O/GCLK3): now also TP65.1
- net ~{Dev_Sel_0} renamed ~{RAM}
- new net: Jx2.3 (Pin_3), R96.1
- new net: TP58.1, U3.29 (I/O)
- new net: TP54.1, U2.45 (I/O)
- new net: TP53.1, U2.46 (I/O)
- new net: R97.1, RomMapped1.2 (A)
- new net: Jx2.1 (Pin_1), R95.1
Other:
- note added: "Dev_Sel_0 = RAM Dev_Sel_1 = OnBoard VIA Dev_Sel_2 = OnBoard ACIA Dev_Sel_3 = Bus_1 Dev_Sel_4 = Bus_2 Dev_Sel_5 = Bus_3 Dev_Sel_6 = Bus_4 Dev_Sel_7 = OnBoard future use"
- note added: "TESTPOINTS"
- note removed: "Dev_Sel_0 = RAM Dev_Sel_1 = OnBoard VIA Dev_Sel_2 = OnBoard ACIA Dev_Sel_3 = Bus_1 Dev_Sel_4 = Bus_2 Dev_Sel_5 = Bus_3 Dev_Sel_6 = OnBoard future use Dev_Sel_7 = OnBoard future use"
- note removed: "TODO"
- note removed: "dev 1 = VIA, nebo tak nejak s bzucakem"

Commit message: Prvni navrh ATF2
Parts:
- added R100, R102, R98, R99: 10k, MHF:R_0805_2012Metric_Pad1.20x1.40mm_HandSolder, symbol MHF:R
Connections:
- net +5V: now also R100.2, R102.2, R98.2, R99.2
- net A_S_16: now also R100.1
- net B_S_16: now also R102.1
- net ~{RAM}: now also R98.1
- net ~{ROM}: now also R99.1
Other:
- note added: "CONFIG"
- note added: "PULLUPS"
- note added: "SYSTEM LEDs"
