File: HW/KiCad/retro-003/retro-003.kicad_pcb (KiCad board)
At the start: 4 copper layers, 100 x 100 mm, 353 parts, among them J1 Conn_02x05_JTAG, J100 x, J101 x, J102 x, J103 x, J104 x, J105 x, J106 x, J12 Reset, J2 Conn_02x05_JTAG, J21 x, J22 x, J3 Serial, J37 x, J38 x, J39 x, J4 SysBus, J40 x, J41 x, J42 x, J43 x, J44 x, J45 x, J46 x, J47 x, J48 x, J49 x, J5 x, J50 x, J51 x, J52 x, J53 x, J54 x, J55 x, J56 x, J57 x, J58 x, J59 x, J6 SysBus, J60 x, J61 x, J62 x, J63 x, J64 x, J65 x, J66 x, J67 x, J68 x, J69 x, J7 Conn_01x16_Pin, J70 x, J71 x, J72 x, J73 x, J74 x, J75 x, J76 x, J77 x, J78 x, J79 x, J8 x, J80 x, J81 x, J82 x, J83 x, J84 x, J85 x, J86 x, J87 x, J88 x, J89 x, J90 x, J91 x, J92 x, J93 x, J94 x, J95 x, J96 x, J97 x, J98 x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

Commit message: ATF3: fits
Parts:
- added R100: 10k, MHF:R_0805_2012Metric_Pad1.20x1.40mm_HandSolder, F.Cu at (133.0, 47.4)
- added R102: 10k, MHF:R_0805_2012Metric_Pad1.20x1.40mm_HandSolder, F.Cu at (133.0, 50.4)
- added R98: 10k, MHF:R_0805_2012Metric_Pad1.20x1.40mm_HandSolder, F.Cu at (133.0, 41.5)
- added R99: 10k, MHF:R_0805_2012Metric_Pad1.20x1.40mm_HandSolder, F.Cu at (133.0, 44.5)
- added TP37: I, MHF:TestPoint_Pad_1.0x1.0mm, F.Cu at (113.1, 51.2)
- added TP38: I, MHF:TestPoint_Pad_1.0x1.0mm, F.Cu at (119.9, 50.6)
- added U15: ATF1508AS-10AU100, Gilhad_footprints:ATF1508-AS_TQFP100_long, F.Cu at (119.7, 69.6)
Connections:
- net /CA0 renamed /A0
- net /CA1 renamed /A1
- net /CA10 renamed /A10
- net /CA11 renamed /A11
- net /CA2 renamed /A2
- net /CA3 renamed /A3
- net /CA4 renamed /A4
- net /CA5 renamed /A5
- net /CA6 renamed /A6
- net /CA7 renamed /A7
- net /CA8 renamed /A8
- net /CA9 renamed /A9
- net /E renamed /Dev_E
- net /GA12 renamed /A12
- net /GA13 renamed /A13
- net /GA14 renamed /A14
- net /GA15 renamed /A15
- net /R~{W} renamed /Dev_R~{W}
- net /mB_HALT renamed /B_HALT
- net /mB_READ renamed /B_READ
- net /mB_SHARE_DIRTY renamed /B_SHARE_DIRTY
- net /mB_SHARE_GRANTED renamed /B_SHARE_GRANTED
- net /mB_SHARE_REQUEST renamed /B_SHARE_REQUEST
- net /mB_SHARE_SELECT renamed /B_SHARE_SELECT
- net /mB_S_16 renamed /B_S_16
- net /~{Dev_Sel_3} renamed /~{Dev_1}
- net /~{Dev_Sel_4} renamed /~{Dev_2}
- net /~{Dev_Sel_5} renamed /~{Dev_3}
- net /~{Dev_Sel_6} renamed /~{Dev_4}
- net /~{FIRQ} renamed /~{Dev_FIRQ}
- net /~{IRQ} renamed /~{Dev_IRQ}
- net /~{NMI} renamed /~{Dev_NMI}

Commit message: Kicad traces, labels
Parts:
- removed L15, L16, L18, L19, L20, L21, L22, L23, L24, L25, L26, L27, L28, L29, L30, L31, L32, L33, L34, L35, LHALT1, LReset1: A0, MHF:LED_0805_2012Metric
- removed R15, R16, R18, R19, R20, R21, R22, R23, R24, R25, R26, R27, R28, R29, R30, R31, R32, R33, R34, R35, R65, R66, R97: 1k, MHF:R_0805_2012Metric_Pad1.20x1.40mm_HandSolder
- removed R67, R68: 4k8, MHF:R_0805_2012Metric_Pad1.20x1.40mm_HandSolder
- removed RomMapped1: RomMapped, MHF:LED_0805_2012Metric
- removed TP49, TP50, TP51, TP52, TP53, TP54, TP55, TP56, TP57, TP58: IO, MHF:TestPoint_Pad_1.0x1.0mm
- removed TP65, TP67, TP70, TP72: I, MHF:TestPoint_Pad_1.0x1.0mm
- removed U10, U11, U9: 74HC14, MHF:SOIC-14_3.9x8.7mm_P1.27mm
- removed U2, U3: ATF1504AS-10AU100, Gilhad_footprints:ATF1504-AS_TQFP100_long
- added JP4: Nx1, MHF:SolderJumper-2_P1.3mm_Bridged_Pad1.0x1.5mm, B.Cu at (206.4, 106.3)
- added JP5: Nx2, MHF:SolderJumper-2_P1.3mm_Bridged_Pad1.0x1.5mm, B.Cu at (206.1, 97.9)
- added TP39: ~{N1}, MHF:TestPoint_Pad_1.0x1.0mm, B.Cu at (206.1, 102.6)
- added TP40: ~{N2}, MHF:TestPoint_Pad_1.0x1.0mm, B.Cu at (201.3, 98.7)
- J1: value Conn_02x05_JTAG -> ATF_JTAG
- J2: value Conn_02x05_JTAG -> Conn_02x04_Top_Bottom; footprint Connector_IDC:IDC-Header_2x05_P2.54mm_Vertical -> Connector_PinSocket_2.54mm:PinSocket_2x04_P2.54mm_Vertical
- L0: value A0 -> LReset
- L1: value A0 -> LHALT
- L10: value A0 -> ACIA
- L11: value A0 -> VIA
- L12: value A0 -> Dev_6
- L13: value A0 -> Dev_5
- L14: value A0 -> Dev_4
- L17: value A0 -> Dev_7
- L2: value A0 -> A_HALT
- L3: value A0 -> ROM
- L37: value A0 -> A1
- L38: value A0 -> A2
- L39: value A0 -> A3
- L4: value A0 -> LRomMapped
- L40: value A0 -> A4
- L41: value A0 -> A5
- L42: value A0 -> A6
- L43: value A0 -> A7
- L5: value A0 -> B_HALT
- L58: value A0 -> Rx
- L59: value A0 -> Tx
- L6: value A0 -> MHF_B
- L7: value A0 -> MHF_A
- L8: value A0 -> RAM
- L9: value A0 -> Dev_3
- LSys1: value A0 -> Sys
- M3, R64: moved to F.Cu
- R100, R102, R60, R63, R93, R98, R99: moved to B.Cu
- R48, R49, R50, R51: value 5k8 -> 10k; footprint Resistor_SMD:R_0805_2012Metric -> MHF:R_0805_2012Metric_Pad1.20x1.40mm_HandSolder; moved to F.Cu
- R52, R54, R55: value 220 -> 10k; footprint Resistor_SMD:R_0805_2012Metric -> MHF:R_0805_2012Metric_Pad1.20x1.40mm_HandSolder; moved to F.Cu
- R53: value 220 -> 10k; footprint Resistor_SMD:R_0805_2012Metric -> MHF:R_0805_2012Metric_Pad1.20x1.40mm_HandSolder
- R56, R57, R58: value 5k8 -> 10k; footprint Resistor_SMD:R_0805_2012Metric -> MHF:R_0805_2012Metric_Pad1.20x1.40mm_HandSolder
- R59: value 5k8 -> 10k; footprint Resistor_SMD:R_0805_2012Metric -> MHF:R_0805_2012Metric_Pad1.20x1.40mm_HandSolder; moved to B.Cu
- TP37: value I -> N1; moved to B.Cu
- TP38: value I -> N2; moved to B.Cu
- moved TP37 107.2 mm to (206.1, 104.3)
- moved TP38 96.8 mm to (203.8, 98.7)
- moved L6 95.8 mm to (189.2, 120.7)
- moved R6 95.8 mm to (189.2, 120.7), turned to 90 degrees
- moved L7 94.6 mm to (186.7, 120.7)
- moved R7 94.6 mm to (186.7, 120.7), turned to 90 degrees
- moved L5 93.1 mm to (174.0, 120.7)
- moved R5 93.1 mm to (174.0, 120.7), turned to 90 degrees
- moved L12 93.0 mm to (207.0, 120.7)
- moved L9 93.0 mm to (199.4, 120.7)
- moved R12 93.0 mm to (207.0, 120.7), turned to 90 degrees
- moved R9 93.0 mm to (199.4, 120.7), turned to 90 degrees
- moved R1 92.9 mm to (165.1, 120.7), turned to 90 degrees
- moved R2 92.9 mm to (167.6, 120.7), turned to 90 degrees
- moved L8 92.8 mm to (184.2, 120.7)
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Connections:
- net /Dev_E renamed /E
- J2 pad 1: Net-(J2-TCK) -> +5V
- J2 pad 3: Net-(J2-TDO) -> +5V
- J2 pad 4: +5V -> GND
- J2 pad 5: Net-(J2-TMS) -> +5V
- J2 pad 6: unconnected-(J2-NC-Pad6) -> GND
- J2 pad 7: unconnected-(J2-NC-Pad7) -> +5V
- J2 pad 8: unconnected-(J2-NC-Pad8) -> GND
- J4 pad 11: /A0 -> /CA0
- J4 pad 12: /A1 -> /CA1
- J4 pad 13: /A2 -> /CA2
- J4 pad 14: /A3 -> /CA3
- J4 pad 15: /A4 -> /CA4
- J4 pad 16: /A5 -> /CA5
- J4 pad 17: /A6 -> /CA6
- J4 pad 18: /A7 -> /CA7
- J4 pad 19: /A8 -> /CA8
- J4 pad 20: /A9 -> /CA9
- J4 pad 21: /A10 -> /CA10
- J4 pad 22: /A11 -> /CA11
- J4 pad 23: /A12 -> /GA12
- J4 pad 24: /A13 -> /GA13
- J4 pad 25: /A14 -> /GA14
- J4 pad 26: /A15 -> /GA15
- J4 pad 28: /B_S_16 -> /mB_S_16
- J4 pad 52: /B_SHARE_SELECT -> /mB_SHARE_SELECT
- J4 pad 54: /Dev_R~{W} -> /R~{W}
- J4 pad 55: /~{Dev_NMI} -> /~{NMI}
- J4 pad 56: /~{Dev_IRQ} -> /~{IRQ}
- J4 pad 57: /~{Dev_FIRQ} -> /~{FIRQ}
- J4 pad 58: /~{Dev_1} -> /~{Dev_Sel_3}
- J4 pad 59: /~{Dev_2} -> /~{Dev_Sel_4}
- J4 pad 60: /~{Dev_3} -> /~{Dev_Sel_5}
- J4 pad 61: /~{Dev_4} -> /~{Dev_Sel_6}
- J6 pad 11: /A0 -> /CA0
- J6 pad 12: /A1 -> /CA1
- J6 pad 13: /A2 -> /CA2
- J6 pad 14: /A3 -> /CA3
- J6 pad 15: /A4 -> /CA4
- J6 pad 16: /A5 -> /CA5
- J6 pad 17: /A6 -> /CA6
- J6 pad 18: /A7 -> /CA7
- J6 pad 19: /A8 -> /CA8
- J6 pad 20: /A9 -> /CA9
- J6 pad 21: /A10 -> /CA10
- J6 pad 22: /A11 -> /CA11
- J6 pad 23: /A12 -> /GA12
- J6 pad 24: /A13 -> /GA13
- J6 pad 25: /A14 -> /GA14
- J6 pad 26: /A15 -> /GA15
- J6 pad 28: /B_S_16 -> /mB_S_16
- J6 pad 52: /B_SHARE_SELECT -> /mB_SHARE_SELECT
- J6 pad 54: /Dev_R~{W} -> /R~{W}
- J6 pad 55: /~{Dev_NMI} -> /~{NMI}
- J6 pad 56: /~{Dev_IRQ} -> /~{IRQ}
- J6 pad 57: /~{Dev_FIRQ} -> /~{FIRQ}
- J6 pad 58: /~{Dev_1} -> /~{Dev_Sel_3}
- J6 pad 59: /~{Dev_2} -> /~{Dev_Sel_4}
- J6 pad 60: /~{Dev_3} -> /~{Dev_Sel_5}
- J6 pad 61: /~{Dev_4} -> /~{Dev_Sel_6}
- L0 pad 1: Net-(L0-K) -> GND
- L0 pad 2: +5V -> Net-(L0-A)
- L1 pad 1: Net-(L1-K) -> GND
- L1 pad 2: +5V -> Net-(L1-A)
- L10 pad 1: Net-(L10-K) -> GND
- L10 pad 2: +5V -> Net-(L10-A)
- L11 pad 1: Net-(L11-K) -> GND
- L11 pad 2: +5V -> Net-(L11-A)
- L12 pad 1: Net-(L12-K) -> GND
- L12 pad 2: +5V -> Net-(L12-A)
- L13 pad 1: Net-(L13-K) -> GND
- L13 pad 2: +5V -> Net-(L13-A)
- L14 pad 1: Net-(L14-K) -> GND
- L14 pad 2: +5V -> Net-(L14-A)
- L17 pad 1: Net-(L17-K) -> +5V
- L17 pad 2: +5V -> Net-(L17-A)
- L2 pad 1: Net-(L2-K) -> GND
- L2 pad 2: +5V -> Net-(L2-A)
- L3 pad 1: Net-(L3-K) -> GND
- L3 pad 2: +5V -> Net-(L3-A)
- L4 pad 1: Net-(L4-K) -> GND
- L4 pad 2: +5V -> Net-(L4-A)
- L5 pad 1: Net-(L5-K) -> GND
- L5 pad 2: +5V -> Net-(L5-A)
- L8 pad 1: Net-(L8-K) -> GND
- L8 pad 2: +5V -> Net-(L8-A)
- L9 pad 1: Net-(L9-K) -> GND
- L9 pad 2: +5V -> Net-(L9-A)
- LSys1 pad 1: GND -> Net-(LSys1-K)
- LSys1 pad 2: Net-(LSys1-A) -> +5V
- M3 pad 1: /A11 -> /CA11
- M3 pad 11: /A14 -> /GA14
- M3 pad 12: /A12 -> /GA12
- M3 pad 13: /A7 -> /CA7
- M3 pad 14: /A6 -> /CA6
- M3 pad 15: /A5 -> /CA5
- M3 pad 16: /A4 -> /CA4
- M3 pad 17: /A3 -> /CA3
- M3 pad 18: /A2 -> /CA2
- M3 pad 19: /A1 -> /CA1
- M3 pad 2: /A9 -> /CA9
- M3 pad 20: /A0 -> /CA0
- M3 pad 3: /A8 -> /CA8
- M3 pad 31: /A10 -> /CA10
- M3 pad 4: /A13 -> /GA13
- M3 pad 7: /A15 -> /GA15
- R0 pad 1: Net-(L0-K) -> Net-(L2-A)
- R1 pad 1: Net-(L1-K) -> Net-(L0-A)
- R10 pad 1: Net-(L10-K) -> Net-(L10-A)
- R102 pad 1: /B_S_16 -> /mB_S_16
- R11 pad 1: Net-(L11-K) -> Net-(L11-A)
- R12 pad 1: Net-(L12-K) -> Net-(L12-A)
- R13 pad 1: Net-(L13-K) -> Net-(L13-A)
- R14 pad 1: Net-(L14-K) -> Net-(L14-A)
- R17 pad 1: Net-(L17-K) -> Net-(L17-A)
- R2 pad 1: Net-(L2-K) -> Net-(L1-A)
- R3 pad 1: Net-(L3-K) -> Net-(L3-A)
- R4 pad 1: Net-(L4-K) -> Net-(L4-A)
- R48 pad 1: JT2_TCK -> /~{NMI}
- R49 pad 1: JT2_TDO -> /~{IRQ}
- R5 pad 1: Net-(L5-K) -> Net-(L5-A)
- R50 pad 1: JT2_TMS -> /~{FIRQ}
- R51 pad 1: JT2_TDI -> ~{DMA/BREQ}
- R52 pad 1: JT2_TCK -> MRDY
- R52 pad 2: Net-(J2-TCK) -> +5V
- R53 pad 1: JT2_TDO -> ~{Dev_Sel_1}
- R53 pad 2: Net-(J2-TDO) -> +5V
- R54 pad 1: JT2_TMS -> ~{Dev_Sel_2}
- R54 pad 2: Net-(J2-TMS) -> +5V
- R55 pad 1: JT2_TDI -> /~{Dev_Sel_3}
- R55 pad 2: Net-(J2-TDI) -> +5V
- R56 pad 1: GND -> /~{Dev_Sel_4}
- R56 pad 2: JT2_TCK -> +5V
- R57 pad 1: GND -> /~{Dev_Sel_5}
- R57 pad 2: JT2_TDO -> +5V
- R58 pad 1: GND -> /~{Dev_Sel_6}
- R58 pad 2: JT2_TMS -> +5V
- R59 pad 1: GND -> ~{Dev_Sel_7}
- R59 pad 2: JT2_TDI -> +5V
- R62 pad 1: Net-(LSys1-A) -> GND
- R62 pad 2: +5V -> Net-(LSys1-K)
- R8 pad 1: Net-(L8-K) -> Net-(L8-A)
- R9 pad 1: Net-(L9-K) -> Net-(L9-A)
- TP37 pad 1: Net-(U15-12V/INPUT/OE1) -> Net-(JP4-B)
- TP38 pad 1: Net-(U15-I/O/GCLK3) -> Net-(JP5-B)
- U1 pad 10: /A2 -> /CA2
- U1 pad 11: /A3 -> /CA3
- U1 pad 12: /A4 -> /CA4
- U1 pad 13: /A5 -> /CA5
- U1 pad 14: /A6 -> /CA6
- U1 pad 15: /A7 -> /CA7
- U1 pad 16: /A8 -> /CA8
- U1 pad 17: /A9 -> /CA9
- U1 pad 18: /A10 -> /CA10
- U1 pad 19: /A11 -> /CA11
- U1 pad 2: /~{Dev_NMI} -> /~{NMI}
- U1 pad 3: /~{Dev_IRQ} -> /~{IRQ}
- U1 pad 32: /Dev_R~{W} -> /R~{W}
- U1 pad 4: /~{Dev_FIRQ} -> /~{FIRQ}
- U1 pad 8: /A0 -> /CA0
- U1 pad 9: /A1 -> /CA1
- U14 pad 1: /A14 -> /GA14
- U14 pad 10: /A0 -> /CA0
- U14 pad 2: /A12 -> /GA12
- U14 pad 21: /A10 -> /CA10
- U14 pad 23: /A11 -> /CA11
- U14 pad 24: /A9 -> /CA9
- U14 pad 25: /A8 -> /CA8
- U14 pad 26: /A13 -> /GA13
- U14 pad 3: /A7 -> /CA7
- U14 pad 4: /A6 -> /CA6
- U14 pad 5: /A5 -> /CA5
- U14 pad 6: /A4 -> /CA4
- U14 pad 7: /A3 -> /CA3
- U14 pad 8: /A2 -> /CA2
- U14 pad 9: /A1 -> /CA1
- U15 pad 1: unconnected-(U15-I/O-Pad1) -> D6
- U15 pad 10: unconnected-(U15-I/O-Pad10) -> /CA5
- U15 pad 100: unconnected-(U15-I/O-Pad100) -> D5
- U15 pad 12: unconnected-(U15-I/O/PD1-Pad12) -> /CA6
- U15 pad 13: unconnected-(U15-I/O-Pad13) -> /CA7
- U15 pad 14: unconnected-(U15-I/O-Pad14) -> /CA8
- U15 pad 16: unconnected-(U15-I/O-Pad16) -> /CA9
- U15 pad 17: unconnected-(U15-I/O-Pad17) -> /CA10
- U15 pad 19: unconnected-(U15-I/O-Pad19) -> /CA11
- U15 pad 2: unconnected-(U15-I/O-Pad2) -> D7
- U15 pad 20: unconnected-(U15-I/O-Pad20) -> CA12
- U15 pad 21: unconnected-(U15-I/O-Pad21) -> CA13
- U15 pad 22: unconnected-(U15-I/O-Pad22) -> CA14
- U15 pad 23: unconnected-(U15-I/O-Pad23) -> CA15
- U15 pad 24: unconnected-(U15-I/O-Pad24) -> /A_S_16
- U15 pad 25: unconnected-(U15-I/O-Pad25) -> /mB_S_16
- U15 pad 27: unconnected-(U15-I/O-Pad27) -> /A_HALT
- U15 pad 28: unconnected-(U15-I/O-Pad28) -> /B_HALT
- U15 pad 29: unconnected-(U15-I/O-Pad29) -> /A_READ
- U15 pad 30: unconnected-(U15-I/O-Pad30) -> /B_READ
- U15 pad 31: unconnected-(U15-I/O-Pad31) -> /A_SHARE_DIRTY
- U15 pad 32: unconnected-(U15-I/O-Pad32) -> /B_SHARE_DIRTY
- U15 pad 33: unconnected-(U15-I/O-Pad33) -> /A_SHARE_GRANTED
- U15 pad 35: unconnected-(U15-I/O-Pad35) -> /B_SHARE_GRANTED
- U15 pad 36: unconnected-(U15-I/O-Pad36) -> /A_SHARE_REQUEST
- U15 pad 37: unconnected-(U15-I/O-Pad37) -> /B_SHARE_REQUEST
- U15 pad 40: unconnected-(U15-I/O-Pad40) -> A_S_SELECT
- U15 pad 41: unconnected-(U15-I/O/PD2-Pad41) -> B_S_SELECT
- U15 pad 42: unconnected-(U15-I/O-Pad42) -> A_S_READ
- U15 pad 44: unconnected-(U15-I/O-Pad44) -> B_S_READ
- U15 pad 45: unconnected-(U15-I/O-Pad45) -> A_S_WRITE
- U15 pad 46: unconnected-(U15-I/O-Pad46) -> B_S_WRITE
- U15 pad 47: unconnected-(U15-I/O-Pad47) -> A_G_ENABLE
- U15 pad 48: unconnected-(U15-I/O-Pad48) -> B_G_ENABLE
- U15 pad 49: unconnected-(U15-I/O-Pad49) -> A_G_A_DIR
- U15 pad 5: unconnected-(U15-I/O-Pad5) -> /CA0
- U15 pad 50: unconnected-(U15-I/O-Pad50) -> B_G_A_DIR
- U15 pad 52: unconnected-(U15-I/O-Pad52) -> A_G_D_DIR
- U15 pad 53: unconnected-(U15-I/O-Pad53) -> B_G_D_DIR
- U15 pad 54: unconnected-(U15-I/O-Pad54) -> /A_SHARE_SELECT
- U15 pad 55: unconnected-(U15-I/O-Pad55) -> /mB_SHARE_SELECT
- U15 pad 56: unconnected-(U15-I/O-Pad56) -> GA16
- U15 pad 57: unconnected-(U15-I/O-Pad57) -> /GA15
- U15 pad 58: unconnected-(U15-I/O-Pad58) -> /GA14
- U15 pad 6: unconnected-(U15-I/O-Pad6) -> /CA1
- U15 pad 60: unconnected-(U15-I/O-Pad60) -> /GA13
- U15 pad 61: unconnected-(U15-I/O-Pad61) -> /GA12
- U15 pad 63: unconnected-(U15-I/O-Pad63) -> ~{Read}
- U15 pad 64: unconnected-(U15-I/O-Pad64) -> ~{Write}
- U15 pad 65: unconnected-(U15-I/O-Pad65) -> ~{ROM}
- U15 pad 67: unconnected-(U15-I/O-Pad67) -> ~{RAM}
- U15 pad 68: unconnected-(U15-I/O-Pad68) -> ~{Dev_Sel_1}
- U15 pad 69: unconnected-(U15-I/O-Pad69) -> ~{Dev_Sel_2}
- U15 pad 7: unconnected-(U15-I/O-Pad7) -> /CA2
- U15 pad 70: unconnected-(U15-I/O-Pad70) -> /~{Dev_Sel_3}
- U15 pad 71: unconnected-(U15-I/O-Pad71) -> /~{Dev_Sel_4}
- U15 pad 72: unconnected-(U15-I/O-Pad72) -> /~{Dev_Sel_5}
- U15 pad 75: unconnected-(U15-I/O-Pad75) -> /~{Dev_Sel_6}
- U15 pad 76: unconnected-(U15-I/O-Pad76) -> ~{Dev_Sel_7}
- U15 pad 77: unconnected-(U15-I/O-Pad77) -> BS
- U15 pad 78: unconnected-(U15-I/O-Pad78) -> MRDY
- U15 pad 79: unconnected-(U15-I/O-Pad79) -> ~{DMA/BREQ}
- U15 pad 8: unconnected-(U15-I/O-Pad8) -> /CA3
- U15 pad 80: unconnected-(U15-I/O-Pad80) -> /~{FIRQ}
- U15 pad 81: unconnected-(U15-I/O-Pad81) -> /~{IRQ}
- U15 pad 83: unconnected-(U15-I/O-Pad83) -> /~{NMI}
- U15 pad 84: unconnected-(U15-I/O-Pad84) -> /BootSrc
- U15 pad 85: Net-(U15-I/O/GCLK3) -> /RomMapped
- U15 pad 88: Net-(U15-12V/INPUT/OE1) -> BA
- U15 pad 9: unconnected-(U15-I/O-Pad9) -> /CA4
- U15 pad 92: unconnected-(U15-I/O-Pad92) -> ~{HALT}
- U15 pad 93: unconnected-(U15-I/O-Pad93) -> /R~{W}
- U15 pad 94: unconnected-(U15-I/O-Pad94) -> D0
- U15 pad 96: unconnected-(U15-I/O-Pad96) -> D1
- U15 pad 97: unconnected-(U15-I/O-Pad97) -> D2
- U15 pad 98: unconnected-(U15-I/O-Pad98) -> D3
- U15 pad 99: unconnected-(U15-I/O-Pad99) -> D4
- U4 pad 11: /A0 -> /CA0
- U4 pad 13: /Dev_R~{W} -> /R~{W}
- U4 pad 7: /~{Dev_IRQ} -> /~{IRQ}
- U5 pad 21: /Dev_R~{W} -> /R~{W}
- U5 pad 35: /A1 -> /CA1
- U5 pad 36: /A0 -> /CA0
- U6 pad 1: D2 -> /A_HALT
- U6 pad 11: D6 -> /RomMapped
- U6 pad 13: D7 -> /B_HALT
- U6 pad 3: D3 -> ~{HALT}
- U6 pad 4: Net-(R1-Pad2) -> Net-(R2-Pad2)
- U6 pad 5: D4 -> MasterReset
- U6 pad 6: Net-(R2-Pad2) -> Net-(R1-Pad2)
- U6 pad 9: D5 -> ~{ROM}
- U7 pad 1: D0 -> /B_SHARE_GRANTED
- U7 pad 11: /A2 -> ~{Dev_Sel_2}
- U7 pad 13: /A3 -> ~{Dev_Sel_1}
- U7 pad 3: D1 -> /A_SHARE_GRANTED
- U7 pad 5: /A0 -> ~{RAM}
- U7 pad 9: /A1 -> /~{Dev_Sel_3}
- U8 pad 1: /A4 -> /~{Dev_Sel_6}
- U8 pad 11: /A8 -> Net-(JP4-B)
- U8 pad 13: /A9 -> ~{Dev_Sel_7}
- U8 pad 3: /A5 -> /~{Dev_Sel_5}
- U8 pad 5: /A6 -> /~{Dev_Sel_4}
- U8 pad 9: /A7 -> Net-(JP5-B)
Routing:
- net /~{Dev_IRQ}: track 226.4 -> 0.00 mm, vias 2 -> 0
- net /A0: track 220.8 -> 0.00 mm, vias 4 -> 0
- net /CA0: track 0.00 -> 191.7 mm, vias 0 -> 3
- net /Dev_R~{W}: track 190.0 -> 0.00 mm, vias 5 -> 0
- net /A1: track 188.4 -> 0.00 mm, vias 4 -> 0
- net /R~{W}: track 0.00 -> 181.4 mm, vias 0 -> 4
- net /~{IRQ}: track 0.00 -> 175.8 mm, vias 0 -> 3
- net /CA1: track 0.00 -> 172.7 mm, vias 0 -> 1
- net /A9: track 156.1 -> 0.00 mm, vias 1 -> 0
- net /A2: track 155.6 -> 0.00 mm, vias 2 -> 0
- net /~{Dev_FIRQ}: track 154.6 -> 0.00 mm, vias 2 -> 0
- net /~{Dev_NMI}: track 152.7 -> 0.00 mm, vias 1 -> 0
- net /A8: track 147.1 -> 0.00 mm, vias 1 -> 0
- net /A11: track 147.0 -> 0.00 mm, vias 1 -> 0
- net /~{Dev_2}: track 145.0 -> 0.00 mm, vias 1 -> 0
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Other:
- board text added: "+5V Gnd"
- board text added: "3 4 5 6 7"
- board text added: "A/B"
- board text added: "Gnd"
- board text added: "Gnd +5V"
- board text added: "HALT A/B"
- board text added: "IN"
- board text added: "Mapped"
- board text added: "OUT"
- board text added: "RAM"
- board text added: "ROM"
- board text added: "Res"

Commit message: PCB finished, ready to be send to JLCpcb
Parts:
- L44: value A0 -> B0
- L45, L55: value A0 -> B1
- L46, L54: value A0 -> B2
- L47: value A0 -> B3
- L48: value A0 -> B4
- L49: value A0 -> B5
- L50: value A0 -> B6
- L51: value A0 -> B7
- L52: value A0 -> IA
- L53: value A0 -> IB
- L56: value A0 -> A2
- L57: value A0 -> A1
- LS1: footprint Buzzer_Beeper:MagneticBuzzer_Kingstate_KCG0601 -> Buzzer_Beeper:Buzzer_12x9.5RM7.6
- R61: moved to B.Cu
- XTAL1: footprint Crystal:Crystal_HC52-6mm_Vertical -> Crystal:Crystal_HC49-4H_Vertical
- moved LS1 40.8 mm to (212.3, 58.6), turned to 0 degrees
- moved Q1 27.6 mm to (218.4, 52.8), turned to -90 degrees
- moved R61 23.6 mm to (220.5, 49.6), turned to 180 degrees
- moved R53 11.2 mm to (221.2, 41.5), turned to -90 degrees
- moved C12 10.9 mm to (210.9, 51.0)
- moved C2 2.85 mm to (219.0, 37.7)
- moved C1 2.81 mm to (219.0, 29.5)
- moved Cx15 2.43 mm to (222.8, 29.0)
- moved XTAL1 1.78 mm to (213.8, 32.2)
- moved R63 1.05 mm to (212.1, 27.0)
- moved L44 0.63 mm to (241.9, 61.6)
- moved L45 0.63 mm to (241.9, 59.1)
- moved L46 0.63 mm to (241.9, 56.5)
- moved L47 0.63 mm to (241.9, 54.0)
- moved L48 0.63 mm to (241.9, 51.4)
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Connections:
- net /A_READ renamed /mA_READ
- net /A_SHARE_GRANTED renamed /mA_SHARE_GRANTED
- net /A_SHARE_SELECT renamed /mA_SHARE_SELECT
- net /B_HALT renamed /mB_HALT
- net /B_SHARE_GRANTED renamed /mB_SHARE_GRANTED
- net /mB_SHARE_SELECT renamed /B_SHARE_SELECT
- net /mB_S_16 renamed /B_S_16
- net /~{Dev_Sel_3} renamed /~{Dev_1}
- net /~{Dev_Sel_4} renamed /~{Dev_2}
- net /~{Dev_Sel_5} renamed /~{Dev_3}
- net /~{Dev_Sel_6} renamed /~{Dev_4}
- L17 pad 1: +5V -> GND
Routing:
- net GND: track 93.8 -> 113.4 mm, vias 49 -> 48
- net ~{Dev_Sel_1}: track 109.1 -> 102.4 mm
- net Net-(U1-EXTAL): track 8.37 -> 12.3 mm
- net Net-(PB1-Pin_8): track 29.2 -> 32.8 mm
- net +5V: track 79.1 -> 82.5 mm, vias 38 -> 36
- net Net-(Q1-C): track 3.72 -> 6.52 mm, vias 0 -> 1
- net Net-(U1-XTAL): track 7.81 -> 10.6 mm
- net MRDY: track 44.2 -> 41.6 mm
- net Net-(L57-A): track 1.81 -> 3.62 mm
- net Net-(L56-A): track 1.81 -> 3.62 mm
- net D6: track 185.7 -> 186.9 mm
- net Net-(Q1-B): track 2.26 -> 3.33 mm, vias 1 -> 0
- net Net-(L6-K): track 3.49 -> 2.65 mm
- net D5: track 180.0 -> 180.8 mm
- net ~{HALT}: track 105.1 -> 105.9 mm
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Other:
- board text added: "115.200 Baud"
- board text added: "2026.08.20"
- board text added: "4 MHz clock"
- board text added: "A/B A16"
- board text added: "A/B halt"
- board text added: "ACIA"
- board text added: "CPU card"
- board text added: "Comp24"
- board text added: "GLUE"
- board text added: "HD6309"
- board text added: "RAM 128kB"
- board text added: "ROM 32kB"
- board text added: "VIA"
- board text added: "Ver. retro-003"
- board text added: "empty"
- board text added: "gilhad@seznam.cz"
- board text added: "https://github.com/githubgilhad/HW-001/tree/master/HW/KiCad/retro-003"
- board text added: "ver. retro-003"
