File: HW/KiCad/retro-003/retro-003.kicad_sch (KiCad schematic)
At the start: 357 parts, among them J1 Conn_02x05_JTAG, J100 x, J101 x, J102 x, J103 x, J104 x, J105 x, J106 x, J12 Reset, J2 Conn_02x05_JTAG, J21 x, J22 x, J3 Serial, J37 x, J38 x, J39 x, J4 SysBus, J40 x, J41 x, J42 x, J43 x, J44 x, J45 x, J46 x, J47 x, J48 x, J49 x, J5 x, J50 x, J51 x, J52 x, J53 x, J54 x, J55 x, J56 x, J57 x, J58 x, J59 x, J6 SysBus, J60 x, J61 x, J62 x, J63 x, J64 x, J65 x, J66 x, J67 x, J68 x, J69 x, J7 Conn_01x16_Pin, J70 x, J71 x, J72 x, J73 x, J74 x, J75 x, J76 x, J77 x, J78 x, J79 x, J8 x, J80 x, J81 x, J82 x, J83 x, J84 x, J85 x, J86 x, J87 x, J88 x, J89 x, J90 x, J91 x, J92 x, J93 x, J94 x, J95 x, J96 x, J97 x, J98 x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

Commit message: ATF3: fits
Parts:
- removed J2: Conn_02x05_JTAG, Connector_IDC:IDC-Header_2x05_P2.54mm_Vertical, symbol PCM_Gilhad_symbols:Conn_02x05_JTAG
- removed R48, R49, R50, R51, R56, R57, R58, R59: 5k8, Resistor_SMD:R_0805_2012Metric, symbol Device:R
- removed R52, R53, R54, R55: 220, Resistor_SMD:R_0805_2012Metric, symbol Device:R
- removed R67, R68: 4k8, MHF:R_0805_2012Metric_Pad1.20x1.40mm_HandSolder, symbol MHF:R
- removed TP49, TP50, TP51, TP52, TP53, TP54, TP55, TP56, TP57, TP58: IO, MHF:TestPoint_Pad_1.0x1.0mm, symbol MHF:TestPoint_Probe
- removed TP65, TP67, TP70, TP72: I, MHF:TestPoint_Pad_1.0x1.0mm, symbol MHF:TestPoint_Probe
- removed U2, U3: ATF1504AS-10AU100, Gilhad_footprints:ATF1504-AS_TQFP100_long, symbol PCM_Gilhad_symbols:ATF1504AS-10AU100-logic
- added R48, R49, R50, R51, R52, R53, R54, R55, R56, R57, R58, R59: 10k, MHF:R_0805_2012Metric_Pad1.20x1.40mm_HandSolder, symbol MHF:R
- added U15: ATF1508AS-10AU100, Gilhad_footprints:ATF1508-AS_TQFP100_long, symbol PCM_Gilhad_symbols:ATF1508AS-10AU100-logic
Connections:
- net +5V: now also R48.2, R49.2, R50.2, R51.2, R52.2, R53.2, R54.2, R55.2, R56.2, R57.2, R58.2, R59.2, U15.18 (VCCIO), U15.3 (VCCIO), U15.34 (VCCIO), U15.39 (VCCINT), U15.51 (VCCIO), U15.66 (VCCIO), U15.82 (VCCIO), U15.91 (VCCINT)
- net BA: now also U15.88 (12V/INPUT/OE1)
- net BS: now also U15.77 (I/O)
- net BootSrc: now also U15.84 (I/O)
- net CA0: now also U15.5 (I/O)
- net CA1: now also U15.6 (I/O)
- net CA10: now also U15.17 (I/O)
- net CA11: now also U15.19 (I/O)
- net CA12: now also U15.20 (I/O)
- net CA13: now also U15.21 (I/O)
- net CA14: now also U15.22 (I/O)
- net CA15: now also U15.23 (I/O)
- net CA2: now also U15.7 (I/O)
- net CA3: now also U15.8 (I/O)
- net CA4: now also U15.9 (I/O)
- net CA5: now also U15.10 (I/O)
- net CA6: now also U15.12 (I/O)
- net CA7: now also U15.13 (I/O)
- net CA8: now also U15.14 (I/O)
- net CA9: now also U15.16 (I/O)
- net D0: now also U15.94 (I/O)
- net D1: now also U15.96 (I/O)
- net D2: now also U15.97 (I/O)
- net D3: now also U15.98 (I/O)
- net D4: now also U15.99 (I/O)
- net D5: now also U15.100 (I/O)
- net D6: now also U15.1 (PD1/I/O)
- net D7: now also U15.2 (I/O)
- net E: now also U15.87 (INPUT/GCLK1)
- net GA12: now also U15.61 (I/O)
- net GA13: now also U15.60 (I/O)
- net GA14: now also U15.58 (I/O)
- net GA15: now also U15.57 (I/O)
- net GA16: now also U15.56 (I/O)
- net GND: now also U15.11 (GND), U15.26 (GND), U15.38 (GND), U15.43 (GND), U15.59 (GND), U15.74 (GND), U15.86 (GND), U15.95 (GND)
- net JT_TCK: now also U15.62 (I/O/TCK)
- net JT_TDI: now also U15.4 (I/O/TDI)
- net JT_TDO: now also U15.73 (I/O/TDO)
- net JT_TMS: now also U15.15 (I/O/TMS)
- net MRDY: now also R52.1, U15.78 (I/O)
- net Q: now also U15.90 (INPUT/OE2/GCLK2)
- net RomMapped: now also U15.85 (I/O/GCLK3)
- net R~{W}: now also U15.93 (I/O)
- net mA_G_A_DIR: now also U15.49 (I/O)
- net mA_G_D_DIR: now also U15.52 (I/O)
- net mA_G_ENABLE: now also U15.47 (I/O)
- net mA_HALT: now also U15.27 (I/O)
- net mA_READ: now also U15.29 (I/O)
- net mA_SHARE_DIRTY: now also U15.31 (I/O)
- net mA_SHARE_GRANTED: now also U15.33 (I/O)
- net mA_SHARE_REQUEST: now also U15.36 (I/O)
- net mA_SHARE_SELECT: now also U15.54 (I/O)
- net mA_S_16: now also U15.24 (I/O)
- net mA_S_READ: now also U15.42 (I/O)
- net mA_S_SELECT: now also U15.40 (I/O)
- net mA_S_WRITE: now also U15.45 (I/O)
- net mB_G_A_DIR: now also U15.50 (I/O)
- net mB_G_D_DIR: now also U15.53 (I/O)
- net mB_G_ENABLE: now also U15.48 (I/O)
- net mB_HALT: now also U15.28 (I/O)
- net mB_READ: now also U15.30 (I/O)
- net mB_SHARE_DIRTY: now also U15.32 (I/O)
- net mB_SHARE_GRANTED: now also U15.35 (I/O)
- net mB_SHARE_REQUEST: now also U15.37 (I/O)
- net mB_SHARE_SELECT: now also U15.55 (I/O)
- net mB_S_16: now also U15.25 (I/O)
- net mB_S_READ: now also U15.44 (I/O)
- net mB_S_SELECT: now also U15.41 (I/O/PD2)
- net mB_S_WRITE: now also U15.46 (I/O)
- net ~{DMA/BREQ}: now also R51.1, U15.79 (I/O)
- net ~{Dev_Sel_1}: now also R53.1, U15.68 (I/O)
- net ~{Dev_Sel_2}: now also R54.1, U15.69 (I/O)
- net ~{Dev_Sel_3}: now also R55.1, U15.70 (I/O)
- net ~{Dev_Sel_4}: now also R56.1, U15.71 (I/O)
- net ~{Dev_Sel_5}: now also R57.1, U15.72 (I/O)
- net ~{Dev_Sel_6}: now also R58.1, U15.75 (I/O)
- net ~{Dev_Sel_7}: now also R59.1, U15.76 (I/O)
- net ~{FIRQ}: now also R50.1, U15.80 (I/O)
- net ~{HALT}: now also U15.92 (I/O)
- net ~{IRQ}: now also R49.1, U15.81 (I/O)
- net ~{NMI}: now also R48.1, U15.83 (I/O)
- net ~{RAM}: now also U15.67 (I/O)
- net ~{RESET}: now also U15.89 (INPUT/GCLR)
- net ~{ROM}: now also U15.65 (I/O)
- net ~{Read}: now also U15.63 (I/O)
- net ~{Write}: now also U15.64 (I/O)
- no-connect marks 80 -> 77
Other:
- note removed: "MR = Memory Region"

Commit message: Kicad traces, labels
Parts:
- removed L15, L16, L18, L19, L20, L21, L22, L23, L24, L25, L26, L27, L28, L29, L30, L31, L32, L33, L34, L35, LHALT1, LReset1: A0, MHF:LED_0805_2012Metric, symbol MHF:LED
- removed R15, R16, R18, R19, R20, R21, R22, R23, R24, R25, R26, R27, R28, R29, R30, R31, R32, R33, R34, R35, R65, R66, R97: 1k, MHF:R_0805_2012Metric_Pad1.20x1.40mm_HandSolder, symbol MHF:R
- removed RomMapped1: RomMapped, MHF:LED_0805_2012Metric, symbol MHF:LED
- removed U10, U11, U9: 74HC14, MHF:SOIC-14_3.9x8.7mm_P1.27mm, symbol MHF:74HC14
- added J2: Conn_02x04_Top_Bottom, Connector_PinSocket_2.54mm:PinSocket_2x04_P2.54mm_Vertical, symbol Connector_Generic:Conn_02x04_Odd_Even
- added JP4: Nx1, MHF:SolderJumper-2_P1.3mm_Bridged_Pad1.0x1.5mm, symbol MHF:SolderJumper_2_Bridged
- added JP5: Nx2, MHF:SolderJumper-2_P1.3mm_Bridged_Pad1.0x1.5mm, symbol MHF:SolderJumper_2_Bridged
- added TP37: N1, MHF:TestPoint_Pad_1.0x1.0mm, symbol MHF:TestPoint_Probe
- added TP38: N2, MHF:TestPoint_Pad_1.0x1.0mm, symbol MHF:TestPoint_Probe
- added TP39: ~{N1}, MHF:TestPoint_Pad_1.0x1.0mm, symbol MHF:TestPoint_Probe
- added TP40: ~{N2}, MHF:TestPoint_Pad_1.0x1.0mm, symbol MHF:TestPoint_Probe
- J1: value Conn_02x05_JTAG -> ATF_JTAG
- L0: renamed from L1; value A0 -> LReset
- L1: renamed from L2; value A0 -> LHALT
- L10: value A0 -> ACIA
- L11: value A0 -> VIA
- L12: value A0 -> Dev_6
- L13: value A0 -> Dev_5
- L14: value A0 -> Dev_4
- L17: value A0 -> Dev_7
- L2: renamed from L0; value A0 -> A_HALT
- L3: value A0 -> ROM
- L37: value A0 -> A1
- L38: value A0 -> A2
- L39: value A0 -> A3
- L4: value A0 -> LRomMapped
- L40: value A0 -> A4
- L41: value A0 -> A5
- L42: value A0 -> A6
- L43: value A0 -> A7
- L5: value A0 -> B_HALT
- L58: value A0 -> Rx
- L59: value A0 -> Tx
- L6: value A0 -> MHF_B
- L7: value A0 -> MHF_A
- L8: value A0 -> RAM
- L9: value A0 -> Dev_3
- LSys1: value A0 -> Sys
Connections:
- net +5V: now also L17.1 (K), LSys1.2 (A), J2.1 (Pin_1), J2.3 (Pin_3), J2.5 (Pin_5), J2.7 (Pin_7); no longer L0.2 (A), L1.2 (A), L10.2 (A), L11.2 (A), L12.2 (A), L13.2 (A), L14.2 (A), L17.2 (A), L2.2 (A), L3.2 (A), L4.2 (A), L5.2 (A), L8.2 (A), L9.2 (A), R62.2
- net A_SHARE_GRANTED: now also U7.3
- net B_SHARE_GRANTED: now also U7.1
- net CA0: no longer U7.5
- net CA1: no longer U7.9
- net CA2: no longer U7.11
- net CA3: no longer U7.13
- net CA4: no longer U8.1
- net CA5: no longer U8.3
- net CA6: no longer U8.5
- net CA7: no longer U8.9
- net CA8: no longer U8.11
- net CA9: no longer U8.13
- net D0: no longer U7.1
- net D1: no longer U7.3
- net D2: no longer U6.1
- net D3: no longer U6.3
- net D4: no longer U6.5
- net D5: no longer U6.9
- net D6: no longer U6.11
- net D7: no longer U6.13
- net GND: now also L0.1 (K), L1.1 (K), L10.1 (K), L11.1 (K), L12.1 (K), L13.1 (K), L14.1 (K), L2.1 (K), L3.1 (K), L4.1 (K), L5.1 (K), L8.1 (K), L9.1 (K), R62.1, J2.2 (Pin_2), J2.4 (Pin_4), J2.6 (Pin_6), J2.8 (Pin_8), JP4.1 (A), JP5.1 (A); no longer LSys1.1 (K)
- net RomMapped: now also U6.11
- net mA_HALT: now also U6.1
- net mB_HALT: now also U6.13
- net ~{Dev_Sel_1}: now also U7.13
- net ~{Dev_Sel_2}: now also U7.11
- net ~{Dev_Sel_3}: now also U7.9
- net ~{Dev_Sel_4}: now also U8.5
- net ~{Dev_Sel_5}: now also U8.3
- net ~{Dev_Sel_6}: now also U8.1
- net ~{Dev_Sel_7}: now also U8.13
- net ~{HALT}: now also U6.3
- net ~{RAM}: now also U7.5
- net ~{RESET}: now also U6.5
- net ~{ROM}: now also U6.9
- net at R4.1: now also L4.2 (A); no longer L4.1 (K)
- net at R0.1: now also L2.2 (A); no longer L2.1 (K)
- net at R5.1: now also L5.2 (A); no longer L5.1 (K)
- net at R14.1: now also L14.2 (A); no longer L14.1 (K)
- net at R10.1: now also L10.2 (A); no longer L10.1 (K)
- net at U6.4: now also R2.2; no longer R1.2
- net at R9.1: now also L9.2 (A); no longer L9.1 (K)
- net at R11.1: now also L11.2 (A); no longer L11.1 (K)
- net at R2.1: now also L1.2 (A); no longer L1.1 (K)
- net at U8.8: now also TP40.1
- net at R1.1: now also L0.2 (A); no longer L0.1 (K)
- net at U8.10: now also TP39.1
- net at R17.1: now also L17.2 (A); no longer L17.1 (K)
- net at U6.6: now also R1.2; no longer R2.2
- net at R13.1: now also L13.2 (A); no longer L13.1 (K)
- net at R8.1: now also L8.2 (A); no longer L8.1 (K)
- net at R3.1: now also L3.2 (A); no longer L3.1 (K)
- net at R12.1: now also L12.2 (A); no longer L12.1 (K)
- new net: LSys1.1 (K), R62.2
- new net: JP4.2 (B), TP37.1, U8.11
- new net: JP5.2 (B), TP38.1, U8.9
Other:
- note removed: "1"
- note removed: "5 E, R/~W ~Reset, ~HALT, BA"
- note removed: "ATF - 2"
- moved on the sheet: L0, L1, L10, L11, L12, L13, L14, L17, L2, L3, L4, L5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

Commit message: PCB finished, ready to be send to JLCpcb
Parts:
- L44: value A0 -> B0
- L45, L55: value A0 -> B1
- L46, L54: value A0 -> B2
- L47: value A0 -> B3
- L48: value A0 -> B4
- L49: value A0 -> B5
- L50: value A0 -> B6
- L51: value A0 -> B7
- L52: value A0 -> IA
- L53: value A0 -> IB
- L56: value A0 -> A2
- L57: value A0 -> A1
- LS1: footprint Buzzer_Beeper:MagneticBuzzer_Kingstate_KCG0601 -> Buzzer_Beeper:Buzzer_12x9.5RM7.6
- XTAL1: footprint Crystal:Crystal_HC52-6mm_Vertical -> Crystal:Crystal_HC49-4H_Vertical
Connections:
- net +5V: no longer L17.1 (K)
- net GND: now also L17.1 (K)
Changed lines of the file:
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@@
 					(size 1.27 1.27)
 				)
+				(hide yes)
 			)
 		)
-		(property "Value" "A0"
+		(property "Value" "A1"
 			(at 844.8675 792.48 0)
 			(effects
@@
 					(size 1.27 1.27)
 				)
-				(hide yes)
 			)
 		)
@@
 	)
 	(symbol
+		(lib_id "power:GND")
+		(at 1082.04 209.55 90)
+		(mirror x)
+		(unit 1)
+		(exclude_from_sim no)
+		(in_bom yes)
+		(on_board yes)
+		(dnp no)
+		(fields_autoplaced yes)
+		(property "Reference" "#PWR040"
+			(at 1088.39 209.55 0)
+			(effects
+				(font
+					(size 1.27 1.27)
+				)
+				(hide yes)
+			)
+		)
+		(property "Value" "GND"
+			(at 1085.85 209.5499 90)
+			(effects
+				(font
+					(size 1.27 1.27)
+				)
+				(justify right)
+			)
+		)
+		(property "Footprint" ""
+			(at 1082.04 209.55 0)
+			(effects
+				(font
+					(size 1.27 1.27)
+				)
+				(hide yes)
+			)
+		)
+		(property "Datasheet" ""
+			(at 1082.04 209.55 0)
+			(effects
+				(font
+					(size 1.27 1.27)
+				)
+				(hide yes)
+			)
+		)
+		(property "Description" ""
+			(at 1082.04 209.55 0)
+			(effects
+				(font
+					(size 1.27 1.27)
+				)
+			)
+		)
+		(pin "1"
+		)
+		(instances
+			(project "retro-003"
+				(path "/64851a36-d60f-4ef2-a652-2faeae5c6012"
+					(reference "#PWR040")
+					(unit 1)
+				)
+			)
+		)
+	)
+	(symbol
 		(lib_id "MHF:Conn_01x01")
 		(at 920.75 91.44 0)
@@
 					(size 1.27 1.27)
 				)
+				(hide yes)
 			)
 		)
-		(property "Value" "A0"
+		(property "Value" "B6"
 			(at 844.8675 758.19 0)
 			(effects
@@
 					(size 1.27 1.27)
 				)
-				(hide yes)
 			)
 		)
@@
 					(size 1.27 1.27)
 				)
+				(hide yes)
 			)
 		)
-		(property "Value" "A0"
+		(property "Value" "B2"
 			(at 844.8675 748.03 0)
 			(effects
@@
 					(size 1.27 1.27)
 				)
-				(hide yes)
 			)
 		)
@@
 					(size 1.27 1.27)
 				)
+				(hide yes)
 			)
 		)
-		(property "Value" "A0"
+		(property "Value" "B4"
 			(at 844.8675 753.11 0)
 			(effects
@@
 					(size 1.27 1.27)
 				)
-				(hide yes)
 			)
 		)
@@
 					(size 1.27 1.27)
 				)
+				(hide yes)
 			)
 		)
-		(property "Value" "A0"
+		(property "Value" "B3"
 			(at 844.8675 750.57 0)
 			(effects
@@
 					(size 1.27 1.27)
 				)
-				(hide yes)
 			)
 		)
@@
 	)
 	(symbol
-		(lib_id "MHF:+5V")
-		(at 1082.04 209.55 270)
-		(unit 1)
-		(exclude_from_sim no)
-		(in_bom yes)
-		(on_board yes)
-		(dnp no)
-		(fields_autoplaced yes)
-		(property "Reference" "#PWR040"
-			(at 1078.23 209.55 0)
-			(effects
-				(font
-					(size 1.27 1.27)
-				)
-				(hide yes)
-			)
-		)
-		(property "Value" "+5V"
-			(at 1085.85 209.5499 90)
-			(effects
-				(font
-					(size 1.27 1.27)
-				)
-				(justify left)
-			)
-		)
-		(property "Footprint" ""
-			(at 1082.04 209.55 0)
-			(effects
-				(font
-					(size 1.27 1.27)
-				)
-				(hide yes)
-			)
-		)
-		(property "Datasheet" ""
-			(at 1082.04 209.55 0)
-			(effects
-				(font
-					(size 1.27 1.27)
-				)
-				(hide yes)
-			)
-		)
-		(property "Description" "Power symbol creates a global label with name \"+5V\""
-			(at 1082.04 209.55 0)
-			(effects
-				(font
-					(size 1.27 1.27)
-				)
-				(hide yes)
-			)
-		)
-		(pin "1"
-		)
-		(instances
-			(project "retro-003"
-				(path "/64851a36-d60f-4ef2-a652-2faeae5c6012"
-					(reference "#PWR040")
-					(unit 1)
-				)
-			)
-		)
-	)
-	(symbol
 		(lib_id "power:GND")
 		(at 99.06 44.45 90)
@@
 					(size 1.27 1.27)
 				)
+				(hide yes)
 			)
 		)
-		(property "Value" "A0"
+		(property "Value" "B5"
 			(at 844.8675 755.65 0)
 			(effects
@@
 					(size 1.27 1.27)
 				)
-				(hide yes)
 			)
 		)
@@
 		(dnp no)
 		(property "Reference" "L44"
-			(at 848.6775 744.22 0)
+			(at 844.8675 742.95 0)
 			(effects
 				(font
 					(size 1.27 1.27)
 				)
+				(hide yes)
 			)
 		)
-		(property "Value" "A0"
+		(property "Value" "B0"
 			(at 844.8675 742.95 0)
 			(effects
@@
 					(size 1.27 1.27)
 				)
-				(hide yes)
 			)
 		)
@@
 			)
 		)
-		(property "Footprint" "Buzzer_Beeper:MagneticBuzzer_Kingstate_KCG0601"
+		(property "Footprint" "Buzzer_Beeper:Buzzer_12x9.5RM7.6"
 			(at 943.991 745.49 0)
 			(effects
@@
 					(size 1.27 1.27)
 				)
+				(hide yes)
 			)
 		)
-		(property "Value" "A0"
+		(property "Value" "IA"
 			(at 844.8675 779.78 0)
 			(effects
@@
 					(size 1.27 1.27)
 				)
-				(hide yes)
 			)
 		)
@@
 					(size 1.27 1.27)
 				)
+				(hide yes)
 			)
 		)
-		(property "Value" "A0"
+		(property "Value" "B2"
 			(at 844.8675 784.86 0)
 			(effects
@@
 					(size 1.27 1.27)
 				)
-				(hide yes)
 			)
 		)
@@
 			)
 		)
-		(property "Footprint" "Crystal:Crystal_HC52-6mm_Vertical"
+		(property "Footprint" "Crystal:Crystal_HC49-4H_Vertical"
 			(at 90.17 317.5 0)
 			(effects
@@
 					(size 1.27 1.27)
 				)
+				(hide yes)
 			)
 		)
-		(property "Value" "A0"
+		(property "Value" "B1"
 			(at 844.8675 745.49 0)
 			(effects
@@
 					(size 1.27 1.27)
 				)
-				(hide yes)
 			)
 		)
@@
 					(size 1.27 1.27)
 				)
+				(hide yes)
 			)
 		)
-		(property "Value" "A0"
+		(property "Value" "IB"
 			(at 844.8675 782.32 0)
 			(effects
@@
 					(size 1.27 1.27)
 				)
-				(hide yes)
 			)
 		)
@@
 					(size 1.27 1.27)
 				)
+				(hide yes)
 			)
 		)
-		(property "Value" "A0"
+		(property "Value" "B7"
 			(at 844.8675 760.73 0)
 			(effects
@@
 					(size 1.27 1.27)
 				)
-				(hide yes)
 			)
 		)
@@
 					(size 1.27 1.27)
 				)
+				(hide yes)
 			)
 		)
-		(property "Value" "A0"
+		(property "Value" "B1"
 			(at 844.8675 787.4 0)
 			(effects
@@
 					(size 1.27 1.27)
 				)
-				(hide yes)
 			)
 		)
@@
 					(size 1.27 1.27)
 				)
+				(hide yes)
 			)
 		)
-		(property "Value" "A0"
+		(property "Value" "A2"
 			(at 844.8675 789.94 0)
 			(effects
@@
 					(size 1.27 1.27)
 				)
-				(hide yes)
 			)
 		)
