File: HW/KiCad/retro-003-simul/retro-003-simul.kicad_sch (KiCad schematic)
At the start: 330 parts, among them J1 AREF, J10 NOTEx, J11 Conn_01x16_Pin, J12 Reset, J15 AREF, J16 XTAL2, J18 XTAL1, J19 AVCC, J2 XTAL1, J3 Serial, J34 NOTE, J35 NOTEx, J4 SysBus, J5 XTAL2, J6 SysBus, J7 Conn_01x16_Pin, J8 AVCC, J9 NOTE, M1 CY7C109D-10ZXI, M2 CY7C109D-10ZXI, M3 CY7C109D-10ZXI, M4 CY7C109D-10ZXI, M5 CY7C109D-10ZXI, Q1 MMBT3904, U1 HD6309, U10 74HC245, U11 74HC245, U12 74HC04, U13 74HC74, U14 28C256, U15 ATF1508AS-10AU100, U16 74HC245, U17 74HC245, U18 74HC245, U19 ATMEGA2560, U2 74HC245, U20 74HC14, U21 74AHC573, U3 ATMEGA2560, U4 MC68B50, U5 6822, U6 74HC14, U7 74HC14, U8 74HC14, U9 74AHC573, Y1 1.8432 MHz, Y2 16 MHz, Y3 16 MHz

Commit message: Snad odladeno az do klasickeho bootu
Parts:
- L3: value ROM -> ROM_Sel
- L8: value RAM -> RAM_Sel
Connections:
- net A_SHARE_DIRTY renamed A_SHARE_COOP
- net B_SHARE_DIRTY renamed B_SHARE_COOP
- net ~{RAM} renamed ~{RAM_Sel}
- net ~{ROM} renamed ~{ROM_Sel}
Other:
- note added: "Dev_0 RAM_Sel"
- note added: "Dev_Sel_0 = RAM_Sel Dev_Sel_1 = OnBoard VIA Dev_Sel_2 = OnBoard ACIA Dev_Sel_3 = Bus_1 Dev_Sel_4 = Bus_2 Dev_Sel_5 = Bus_3 Dev_Sel_6 = Bus_4 Dev_Sel_7 = OnBoard future use"
- note added: "EMS RAM_Sel 8000-9FFF A000-BFFFF (shared between Arduino and HD6309)"
- note added: "External RAM_Sel for Arduino"
- note added: "RAM_Sel"
- note added: "ROM_Sel"
- note removed: "Dev_0 RAM"
- note removed: "Dev_Sel_0 = RAM Dev_Sel_1 = OnBoard VIA Dev_Sel_2 = OnBoard ACIA Dev_Sel_3 = Bus_1 Dev_Sel_4 = Bus_2 Dev_Sel_5 = Bus_3 Dev_Sel_6 = Bus_4 Dev_Sel_7 = OnBoard future use"
- note removed: "EMS RAM 8000-9FFF A000-BFFFF (shared between Arduino and HD6309)"
- note removed: "External RAM for Arduino"
- note removed: "RAM"
Changed lines of the file:
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@@
 		)
 	)
-	(text "RAM"
+	(text "RAM_Sel"
 		(exclude_from_sim no)
 		(at 549.91 621.03 0)
@@
 		)
 	)
-	(text "External RAM for Arduino"
+	(text "External RAM_Sel for Arduino"
 		(exclude_from_sim no)
 		(at 1659.89 173.99 0)
@@
 		)
 	)
-	(text "Dev_0 RAM"
+	(text "Dev_0 RAM_Sel"
 		(exclude_from_sim no)
 		(at 567.69 759.46 0)
@@
 		)
 	)
-	(text "External RAM for Arduino"
+	(text "External RAM_Sel for Arduino"
 		(exclude_from_sim no)
 		(at 151.13 177.8 0)
@@
 		)
 	)
-	(text "ROM"
+	(text "ROM_Sel"
 		(exclude_from_sim no)
 		(at 1049.02 635 0)
@@
 		)
 	)
-	(text "EMS\nRAM 8000-9FFF A000-BFFFF\n(shared between Arduino and HD6309)"
+	(text "EMS\nRAM_Sel 8000-9FFF A000-BFFFF\n(shared between Arduino and HD6309)"
 		(exclude_from_sim no)
 		(at 1178.56 265.43 0)
@@
 		)
 	)
-	(text "EMS\nRAM 8000-9FFF A000-BFFFF\n(shared between Arduino and HD6309)"
+	(text "EMS\nRAM_Sel 8000-9FFF A000-BFFFF\n(shared between Arduino and HD6309)"
 		(exclude_from_sim no)
 		(at 632.46 269.24 0)
@@
 		)
 	)
-	(text "Dev_Sel_0 = RAM\nDev_Sel_1 = OnBoard VIA\nDev_Sel_2 = OnBoard ACIA\n\nDev_Sel_3 = Bus_1\nDev_Sel_4 = Bus_2\nDev_Sel_5 = Bus_3\nDev_Sel_6 = Bus_4\n\nDev_Sel_7 = OnBoard future use"
+	(text "Dev_Sel_0 = RAM_Sel\nDev_Sel_1 = OnBoard VIA\nDev_Sel_2 = OnBoard ACIA\n\nDev_Sel_3 = Bus_1\nDev_Sel_4 = Bus_2\nDev_Sel_5 = Bus_3\nDev_Sel_6 = Bus_4\n\nDev_Sel_7 = OnBoard future use"
 		(exclude_from_sim no)
 		(at 966.47 426.72 0)
@@
 		)
 	)
-	(text_box "Native RAM 32K"
+	(text_box "Native RAM_Sel 32K"
 		(exclude_from_sim no)
 		(at 360.68 688.6354 0)
@@
 		)
 	)
-	(text_box "Native RAM ~ ROM 23.75K"
+	(text_box "Native RAM_Sel ~ ROM_Sel 23.75K"
 		(exclude_from_sim no)
 		(at 360.68 676.91 0)
@@
 		)
 	)
-	(label "~{ROM}"
+	(label "~{ROM_Sel}"
 		(at 1384.3 523.24 180)
 		(effects
@@
 		)
 	)
-	(label "B_SHARE_DIRTY"
+	(label "B_SHARE_COOP"
 		(at 857.25 429.26 180)
 		(effects
@@
 		)
 	)
-	(label "~{RAM}"
+	(label "~{RAM_Sel}"
 		(at 1066.8 585.47 0)
 		(effects
@@
 		)
 	)
-	(label "A_SHARE_DIRTY"
+	(label "A_SHARE_COOP"
 		(at 857.25 426.72 180)
 		(effects
@@
 		)
 	)
-	(label "B_SHARE_DIRTY"
+	(label "B_SHARE_COOP"
 		(at 1041.4 196.85 0)
 		(effects
@@
 		)
 	)
-	(label "~{RAM}"
+	(label "~{RAM_Sel}"
 		(at 1384.3 537.21 180)
 		(effects
@@
 		)
 	)
-	(label "B_SHARE_DIRTY"
+	(label "B_SHARE_COOP"
 		(at 109.22 566.42 180)
 		(effects
@@
 		)
 	)
-	(label "B_SHARE_DIRTY"
+	(label "B_SHARE_COOP"
 		(at 989.33 82.55 180)
 		(effects
@@
 		)
 	)
-	(label "~{RAM}"
+	(label "~{RAM_Sel}"
 		(at 948.69 431.8 0)
 		(effects
@@
 		)
 	)
-	(label "A_SHARE_DIRTY"
+	(label "A_SHARE_COOP"
 		(at 269.24 566.42 0)
 		(effects
@@
 		)
 	)
-	(label "A_SHARE_DIRTY"
+	(label "A_SHARE_COOP"
 		(at 824.23 83.82 0)
 		(effects
@@
 		)
 	)
-	(label "~{ROM}"
+	(label "~{ROM_Sel}"
 		(at 948.69 434.34 0)
 		(effects
@@
 		)
 	)
-	(label "A_SHARE_DIRTY"
+	(label "A_SHARE_COOP"
 		(at 664.21 104.14 180)
 		(effects
@@
 		)
 	)
-	(label "RAM"
+	(label "RAM_Sel"
 		(at 154.94 469.9 0)
 		(effects
@@
 		)
 	)
-	(label "B_SHARE_DIRTY"
+	(label "B_SHARE_COOP"
 		(at 894.08 83.82 180)
 		(effects
@@
 		)
 	)
-	(label "ROM"
+	(label "ROM_Sel"
 		(at 191.77 469.9 0)
 		(effects
@@
 		)
 	)
-	(label "B_SHARE_DIRTY"
+	(label "B_SHARE_COOP"
 		(at 1094.74 196.85 180)
 		(effects
@@
 		)
 	)
-	(label "A_SHARE_DIRTY"
+	(label "A_SHARE_COOP"
 		(at 919.48 82.55 0)
 		(effects
@@
 		)
 	)
-	(label "A_SHARE_DIRTY"
+	(label "A_SHARE_COOP"
 		(at 1154.43 105.41 0)
 		(effects
@@
 		)
 	)
-	(label "B_SHARE_DIRTY"
+	(label "B_SHARE_COOP"
 		(at 590.55 104.14 0)
 		(effects
@@
 		)
 	)
-	(label "B_SHARE_DIRTY"
+	(label "B_SHARE_COOP"
 		(at 1228.09 105.41 180)
 		(effects
@@
 		)
 	)
-	(label "A_SHARE_DIRTY"
+	(label "A_SHARE_COOP"
 		(at 1094.74 137.16 180)
 		(effects
@@
 		)
 	)
-	(label "A_SHARE_DIRTY"
+	(label "A_SHARE_COOP"
 		(at 1041.4 137.16 0)
 		(effects
@@
 		)
 	)
-	(label "~{ROM}"
+	(label "~{ROM_Sel}"
 		(at 1062.99 693.42 180)
 		(effects
@@
 		)
 	)
-	(label "~{ROM}"
+	(label "~{ROM_Sel}"
 		(at 468.63 53.34 180)
 		(effects
@@
 		)
 	)
-	(label "~{RAM}"
+	(label "~{RAM_Sel}"
 		(at 468.63 55.88 180)
 		(effects
@@
 		)
 	)
-	(global_label "B_SHARE_DIRTY"
+	(global_label "B_SHARE_COOP"
 		(shape input)
 		(at 629.92 78.74 90)
@@
 		)
 	)
-	(global_label "A_SHARE_DIRTY"
+	(global_label "A_SHARE_COOP"
 		(shape input)
 		(at 1385.57 269.24 0)
@@
 		)
 	)
-	(global_label "B_SHARE_DIRTY"
+	(global_label "B_SHARE_COOP"
 		(shape input)
 		(at 425.45 273.05 180)
@@
 		)
 	)
-	(global_label "A_SHARE_DIRTY"
+	(global_label "A_SHARE_COOP"
 		(shape input)
 		(at 1188.72 80.01 90)
@@
 			)
 		)
-		(property "Value" "RAM"
+		(property "Value" "RAM_Sel"
 			(at 1436.6875 534.67 0)
 			(effects
@@
 			)
 		)
-		(property "Value" "ROM"
+		(property "Value" "ROM_Sel"
 			(at 1436.6875 520.7 0)
 			(effects
